Commit message: Add multi-robot GLB preview and unify Gripper G2 naming.
Extend Genesis visual preview to Lite6, UF850, and xArm5/7 with shared
gripper_g2 and bio_gripper assets; rename user-facing CLI/API to
--gripper-g2 and --bio-gripper-g2; simplify README around view_robot_glb.py.

Co-authored-by: Cursor <cursoragent@cursor.com>

File: assets/urdf/xarm6/xarm6_1305_g2_visual.urdf (robot description, URDF)
Before this commit: robot xarm6_1305_g2_visual, 18 links, 17 joints
Links:
- link gripper_g2_visual: geometry visual mesh filename=../gripper_g2/meshes/visual/gripper_g2_static_link6.glb
- link left_finger: geometry collision mesh filename=../gripper_g2/meshes/collision/left_finger.STL
- link left_inner_knuckle: geometry collision mesh filename=../gripper_g2/meshes/collision/left_inner_knuckle.STL
- link left_outer_knuckle: geometry collision mesh filename=../gripper_g2/meshes/collision/left_outer_knuckle.STL
- link right_finger: geometry collision mesh filename=../gripper_g2/meshes/collision/right_finger.STL
- link right_inner_knuckle: geometry collision mesh filename=../gripper_g2/meshes/collision/right_inner_knuckle.STL
- link right_outer_knuckle: geometry collision mesh filename=../gripper_g2/meshes/collision/right_outer_knuckle.STL
- link xarm_gripper_base_link: geometry collision mesh filename=../gripper_g2/meshes/collision/base_link.STL
Joints:
- joint gripper_fix: parent link_eef -> link6
- joint gripper_g2_visual_fix: parent link_eef -> link6

File: assets/urdf/xarm6/xarm6_with_gripper.urdf (robot description, URDF)
Before this commit: robot xarm6_with_gripper, 17 links, 16 joints
Links:
- link left_finger: geometry collision mesh filename=../gripper_g2/meshes/collision/left_finger.STL; visual mesh filename=../gripper_g2/meshes/collision/left_finger.STL
- link left_inner_knuckle: geometry collision mesh filename=../gripper_g2/meshes/collision/left_inner_knuckle.STL; visual mesh filename=../gripper_g2/meshes/collision/left_inner_knuckle.STL
- link left_outer_knuckle: geometry collision mesh filename=../gripper_g2/meshes/collision/left_outer_knuckle.STL; visual mesh filename=../gripper_g2/meshes/collision/left_outer_knuckle.STL
- link right_finger: geometry collision mesh filename=../gripper_g2/meshes/collision/right_finger.STL; visual mesh filename=../gripper_g2/meshes/collision/right_finger.STL
- link right_inner_knuckle: geometry collision mesh filename=../gripper_g2/meshes/collision/right_inner_knuckle.STL; visual mesh filename=../gripper_g2/meshes/collision/right_inner_knuckle.STL
- link right_outer_knuckle: geometry collision mesh filename=../gripper_g2/meshes/collision/right_outer_knuckle.STL; visual mesh filename=../gripper_g2/meshes/collision/right_outer_knuckle.STL
- link xarm_gripper_base_link: geometry collision mesh filename=../gripper_g2/meshes/collision/base_link.STL; visual mesh filename=../gripper_g2/meshes/collision/base_link.STL
