Commit message: Prepare v0.1.0 public release
- Add multi-robot API exports (ROBOT_PROFILES, paths, kinematics, GLB)
- Fix hardcoded local paths in vendor script and docs
- Remove duplicate .STL files and orphan collision meshes
- Add CONTRIBUTING.md, CHANGELOG.md, CODE_OF_CONDUCT.md
- Add py.typed marker and pyproject.toml metadata
- Expand README with badges, API reference, and contribution guide
- Add asset pipeline READMEs under assets/ and scripts/

Co-Authored-By: Claude <noreply@anthropic.com>

File: assets/urdf/gripper_g2/gripper_g2.urdf (robot description, URDF)
Before this commit: robot gripper_g2, 9 links, 9 joints
Links:
- removed link link_tool
- link left_finger: geometry collision mesh filename=meshes/gripper/xarm/left_finger.stl; visual mesh filename=meshes/gripper/xarm/left_finger.stl
- link left_inner_knuckle: mass 0.023013 -> 0.0230125781256706; geometry collision mesh filename=meshes/gripper/xarm/left_inner_knuckle.stl; visual mesh filename=meshes/gripper/xarm/left_inner_knuckle.stl
- link left_outer_knuckle: geometry collision mesh filename=meshes/gripper/xarm/left_outer_knuckle.stl; visual mesh filename=meshes/gripper/xarm/left_outer_knuckle.stl
- link right_finger: geometry collision mesh filename=meshes/gripper/xarm/right_finger.stl; visual mesh filename=meshes/gripper/xarm/right_finger.stl
- link right_inner_knuckle: geometry collision mesh filename=meshes/gripper/xarm/right_inner_knuckle.stl; visual mesh filename=meshes/gripper/xarm/right_inner_knuckle.stl
- link right_outer_knuckle: geometry collision mesh filename=meshes/gripper/xarm/right_outer_knuckle.stl; visual mesh filename=meshes/gripper/xarm/right_outer_knuckle.stl
- link xarm_gripper_base_link: geometry collision mesh filename=meshes/gripper/xarm/base_link.stl; visual mesh filename=meshes/gripper/xarm/base_link.stl
Joints:
- removed joint gripper_attach
- joint gripper_fix: parent link_eef -> link_tool

File: assets/urdf/uf850/uf850_bio_gripper_visual.glb.urdf (robot description, URDF)
Before this commit: robot uf850_bio_gripper_visual.glb, 9 links, 8 joints
Links:
- added link bio_gripper_base_link, mass 0.38837; collision mesh filename=../bio_gripper/meshes/visual/link_base.stl
- added link bio_gripper_left_finger, mass 0.012105; collision mesh filename=../bio_gripper/meshes/visual/left_finger.stl
- added link bio_gripper_right_finger, mass 0.012068; collision mesh filename=../bio_gripper/meshes/visual/right_finger.stl
- added link link_tcp
Joints:
- added joint bio_gripper_attach: type fixed, parent link6, child bio_gripper_base_link, origin xyz=0 0 0 rpy=0 0 0
- added joint joint_tcp: type fixed, parent bio_gripper_base_link, child link_tcp, origin xyz=0.135 0 0.055 rpy=0 0 0
- added joint left_finger_joint: type prismatic, parent bio_gripper_base_link, child bio_gripper_left_finger, origin xyz=0.059 0 0.027 rpy=0 0 0, axis 0 1 0, limit lower=-0.04 upper=0.0 effort=2.0 velocity=0.1, mimic joint=right_finger_joint multiplier=-1 offset=0
- added joint right_finger_joint: type prismatic, parent bio_gripper_base_link, child bio_gripper_right_finger, origin xyz=0.059 0 0.027 rpy=0 0 0, axis 0 1 0, limit lower=0 upper=0.04 effort=2.0 velocity=0.1

File: assets/urdf/xarm5/xarm5_1305_bio_gripper_visual.glb.urdf (robot description, URDF)
Before this commit: robot xarm5_1305_bio_gripper_visual.glb, 8 links, 7 joints
Links:
- added link bio_gripper_base_link, mass 0.38837; collision mesh filename=../bio_gripper/meshes/visual/link_base.stl
- added link bio_gripper_left_finger, mass 0.012105; collision mesh filename=../bio_gripper/meshes/visual/left_finger.stl
- added link bio_gripper_right_finger, mass 0.012068; collision mesh filename=../bio_gripper/meshes/visual/right_finger.stl
- added link link_tcp
Joints:
- added joint bio_gripper_attach: type fixed, parent link5, child bio_gripper_base_link, origin xyz=0 0 0 rpy=0 0 0
- added joint joint_tcp: type fixed, parent bio_gripper_base_link, child link_tcp, origin xyz=0.135 0 0.055 rpy=0 0 0
- added joint left_finger_joint: type prismatic, parent bio_gripper_base_link, child bio_gripper_left_finger, origin xyz=0.059 0 0.027 rpy=0 0 0, axis 0 1 0, limit lower=-0.04 upper=0.0 effort=2.0 velocity=0.1, mimic joint=right_finger_joint multiplier=-1 offset=0
- added joint right_finger_joint: type prismatic, parent bio_gripper_base_link, child bio_gripper_right_finger, origin xyz=0.059 0 0.027 rpy=0 0 0, axis 0 1 0, limit lower=0 upper=0.04 effort=2.0 velocity=0.1

File: assets/urdf/xarm6/xarm6_1305_bio_gripper_visual.glb.urdf (robot description, URDF)
Before this commit: robot xarm6_1305_bio_gripper_visual.glb, 10 links, 9 joints
Links:
- added link bio_gripper_base_link, mass 0.38837; collision mesh filename=../bio_gripper/meshes/visual/link_base.stl
- added link bio_gripper_left_finger, mass 0.012105; collision mesh filename=../bio_gripper/meshes/visual/left_finger.stl
- added link bio_gripper_right_finger, mass 0.012068; collision mesh filename=../bio_gripper/meshes/visual/right_finger.stl
- added link link_tcp
Joints:
- added joint bio_gripper_attach: type fixed, parent link6, child bio_gripper_base_link, origin xyz=0 0 0 rpy=0 0 0
- added joint joint_tcp: type fixed, parent bio_gripper_base_link, child link_tcp, origin xyz=0.135 0 0.055 rpy=0 0 0
- added joint left_finger_joint: type prismatic, parent bio_gripper_base_link, child bio_gripper_left_finger, origin xyz=0.059 0 0.027 rpy=0 0 0, axis 0 1 0, limit lower=-0.04 upper=0.0 effort=2.0 velocity=0.1, mimic joint=right_finger_joint multiplier=-1 offset=0
- added joint right_finger_joint: type prismatic, parent bio_gripper_base_link, child bio_gripper_right_finger, origin xyz=0.059 0 0.027 rpy=0 0 0, axis 0 1 0, limit lower=0 upper=0.04 effort=2.0 velocity=0.1

File: assets/urdf/xarm7/xarm7_1305_bio_gripper_visual.glb.urdf (robot description, URDF)
Before this commit: robot xarm7_1305_bio_gripper_visual.glb, 10 links, 9 joints
Links:
- added link bio_gripper_base_link, mass 0.38837; collision mesh filename=../bio_gripper/meshes/visual/link_base.stl
- added link bio_gripper_left_finger, mass 0.012105; collision mesh filename=../bio_gripper/meshes/visual/left_finger.stl
- added link bio_gripper_right_finger, mass 0.012068; collision mesh filename=../bio_gripper/meshes/visual/right_finger.stl
- added link link_tcp
Joints:
- added joint bio_gripper_attach: type fixed, parent link7, child bio_gripper_base_link, origin xyz=0 0 0 rpy=0 0 0
- added joint joint_tcp: type fixed, parent bio_gripper_base_link, child link_tcp, origin xyz=0.135 0 0.055 rpy=0 0 0
- added joint left_finger_joint: type prismatic, parent bio_gripper_base_link, child bio_gripper_left_finger, origin xyz=0.059 0 0.027 rpy=0 0 0, axis 0 1 0, limit lower=-0.04 upper=0.0 effort=2.0 velocity=0.1, mimic joint=right_finger_joint multiplier=-1 offset=0
- added joint right_finger_joint: type prismatic, parent bio_gripper_base_link, child bio_gripper_right_finger, origin xyz=0.059 0 0.027 rpy=0 0 0, axis 0 1 0, limit lower=0 upper=0.04 effort=2.0 velocity=0.1
