Commit message: Unify calibrated G2 control and simplify simulation acceptance
Encode the nominal 0-84 mm G2 stroke directly in all 11 standard URDFs,
share geometric conversions across scalar and Torch paths, and remove
runtime model derivation.

Use calibrated G2 controllers across manipulation, viewers and RL;
keep artifact compatibility checks and fail commands on transport rejection.
Consolidate G2 tests into seven files with 22 GPU acceptance cases.

Replace Lite6 link-wide exemptions with geometry-pair collision filters,
update simulation dependencies, and synchronize bilingual documentation.

Validation: project-check fast passed (996 passed, 1 skipped; 81.58%
coverage), 61 safety tests and 41 focused CLI/packaging tests passed.
The preceding 22 GPU cases and CPU transport regression passed; recorded
manipulation results also satisfy the corrected command acceptance gates.

File: assets/urdf/gripper_g2/gripper_g2.urdf (robot description, URDF)
Before this commit: robot gripper_g2, 8 links, 8 joints
Joints:
- joint drive_joint: limit lower=0 upper=0.85 effort=50 velocity=2 -> lower=0.057210812728026743 upper=0.86509464599328212 effort=50 velocity=2.608067454724
- joint left_finger_joint: limit lower=0 upper=0.85 effort=50 velocity=2 -> lower=0.057210812728026743 upper=0.86509464599328212 effort=50 velocity=2.608067454724
- joint left_inner_knuckle_joint: limit lower=0 upper=0.85 effort=50 velocity=2 -> lower=0.057210812728026743 upper=0.86509464599328212 effort=50 velocity=2.608067454724
- joint right_finger_joint: limit lower=0 upper=0.85 effort=50 velocity=2 -> lower=0.057210812728026743 upper=0.86509464599328212 effort=50 velocity=2.608067454724
- joint right_inner_knuckle_joint: limit lower=0 upper=0.85 effort=50 velocity=2 -> lower=0.057210812728026743 upper=0.86509464599328212 effort=50 velocity=2.608067454724
- joint right_outer_knuckle_joint: limit lower=0 upper=0.85 effort=50 velocity=2 -> lower=0.057210812728026743 upper=0.86509464599328212 effort=50 velocity=2.608067454724

File: assets/urdf/gripper_g2/gripper_g2_movable_visual.urdf (robot description, URDF)
Before this commit: robot gripper_g2_movable_visual, 9 links, 8 joints
Joints:
- joint drive_joint: limit lower=0 upper=0.85 effort=50 velocity=2 -> lower=0.057210812728026743 upper=0.86509464599328212 effort=50 velocity=2.608067454724
- joint left_finger_joint: limit lower=0 upper=0.85 effort=50 velocity=2 -> lower=0.057210812728026743 upper=0.86509464599328212 effort=50 velocity=2.608067454724
- joint left_inner_knuckle_joint: limit lower=0 upper=0.85 effort=50 velocity=2 -> lower=0.057210812728026743 upper=0.86509464599328212 effort=50 velocity=2.608067454724
- joint right_finger_joint: limit lower=0 upper=0.85 effort=50 velocity=2 -> lower=0.057210812728026743 upper=0.86509464599328212 effort=50 velocity=2.608067454724
- joint right_inner_knuckle_joint: limit lower=0 upper=0.85 effort=50 velocity=2 -> lower=0.057210812728026743 upper=0.86509464599328212 effort=50 velocity=2.608067454724
- joint right_outer_knuckle_joint: limit lower=0 upper=0.85 effort=50 velocity=2 -> lower=0.057210812728026743 upper=0.86509464599328212 effort=50 velocity=2.608067454724

File: assets/urdf/uf850/uf850_g2_movable_visual.urdf (robot description, URDF)
Before this commit: robot uf850_g2_movable_visual, 16 links, 15 joints
Joints:
- joint drive_joint: limit lower=0 upper=0.85 effort=50 velocity=2 -> lower=0.057210812728026743 upper=0.86509464599328212 effort=50 velocity=2.608067454724
- joint left_finger_joint: limit lower=0 upper=0.85 effort=50 velocity=2 -> lower=0.057210812728026743 upper=0.86509464599328212 effort=50 velocity=2.608067454724
- joint left_inner_knuckle_joint: limit lower=0 upper=0.85 effort=50 velocity=2 -> lower=0.057210812728026743 upper=0.86509464599328212 effort=50 velocity=2.608067454724
- joint right_finger_joint: limit lower=0 upper=0.85 effort=50 velocity=2 -> lower=0.057210812728026743 upper=0.86509464599328212 effort=50 velocity=2.608067454724
- joint right_inner_knuckle_joint: limit lower=0 upper=0.85 effort=50 velocity=2 -> lower=0.057210812728026743 upper=0.86509464599328212 effort=50 velocity=2.608067454724
- joint right_outer_knuckle_joint: limit lower=0 upper=0.85 effort=50 velocity=2 -> lower=0.057210812728026743 upper=0.86509464599328212 effort=50 velocity=2.608067454724

File: assets/urdf/uf850/uf850_g2_visual.urdf (robot description, URDF)
Before this commit: robot uf850_g2_visual, 17 links, 16 joints
Joints:
- joint drive_joint: limit lower=0 upper=0.85 effort=50 velocity=2 -> lower=0.057210812728026743 upper=0.86509464599328212 effort=50 velocity=2.608067454724
- joint left_finger_joint: limit lower=0 upper=0.85 effort=50 velocity=2 -> lower=0.057210812728026743 upper=0.86509464599328212 effort=50 velocity=2.608067454724
- joint left_inner_knuckle_joint: limit lower=0 upper=0.85 effort=50 velocity=2 -> lower=0.057210812728026743 upper=0.86509464599328212 effort=50 velocity=2.608067454724
- joint right_finger_joint: limit lower=0 upper=0.85 effort=50 velocity=2 -> lower=0.057210812728026743 upper=0.86509464599328212 effort=50 velocity=2.608067454724
- joint right_inner_knuckle_joint: limit lower=0 upper=0.85 effort=50 velocity=2 -> lower=0.057210812728026743 upper=0.86509464599328212 effort=50 velocity=2.608067454724
- joint right_outer_knuckle_joint: limit lower=0 upper=0.85 effort=50 velocity=2 -> lower=0.057210812728026743 upper=0.86509464599328212 effort=50 velocity=2.608067454724

File: assets/urdf/xarm5/xarm5_1305_g2_movable_visual.urdf (robot description, URDF)
Before this commit: robot xarm5_1305_g2_movable_visual, 15 links, 14 joints
Joints:
- joint drive_joint: limit lower=0 upper=0.85 effort=50 velocity=2 -> lower=0.057210812728026743 upper=0.86509464599328212 effort=50 velocity=2.608067454724
- joint left_finger_joint: limit lower=0 upper=0.85 effort=50 velocity=2 -> lower=0.057210812728026743 upper=0.86509464599328212 effort=50 velocity=2.608067454724
- joint left_inner_knuckle_joint: limit lower=0 upper=0.85 effort=50 velocity=2 -> lower=0.057210812728026743 upper=0.86509464599328212 effort=50 velocity=2.608067454724
- joint right_finger_joint: limit lower=0 upper=0.85 effort=50 velocity=2 -> lower=0.057210812728026743 upper=0.86509464599328212 effort=50 velocity=2.608067454724
- joint right_inner_knuckle_joint: limit lower=0 upper=0.85 effort=50 velocity=2 -> lower=0.057210812728026743 upper=0.86509464599328212 effort=50 velocity=2.608067454724
- joint right_outer_knuckle_joint: limit lower=0 upper=0.85 effort=50 velocity=2 -> lower=0.057210812728026743 upper=0.86509464599328212 effort=50 velocity=2.608067454724

File: assets/urdf/xarm5/xarm5_1305_g2_visual.urdf (robot description, URDF)
Before this commit: robot xarm5_1305_g2_visual, 16 links, 15 joints
Joints:
- joint drive_joint: limit lower=0 upper=0.85 effort=50 velocity=2 -> lower=0.057210812728026743 upper=0.86509464599328212 effort=50 velocity=2.608067454724
- joint left_finger_joint: limit lower=0 upper=0.85 effort=50 velocity=2 -> lower=0.057210812728026743 upper=0.86509464599328212 effort=50 velocity=2.608067454724
- joint left_inner_knuckle_joint: limit lower=0 upper=0.85 effort=50 velocity=2 -> lower=0.057210812728026743 upper=0.86509464599328212 effort=50 velocity=2.608067454724
- joint right_finger_joint: limit lower=0 upper=0.85 effort=50 velocity=2 -> lower=0.057210812728026743 upper=0.86509464599328212 effort=50 velocity=2.608067454724
- joint right_inner_knuckle_joint: limit lower=0 upper=0.85 effort=50 velocity=2 -> lower=0.057210812728026743 upper=0.86509464599328212 effort=50 velocity=2.608067454724
- joint right_outer_knuckle_joint: limit lower=0 upper=0.85 effort=50 velocity=2 -> lower=0.057210812728026743 upper=0.86509464599328212 effort=50 velocity=2.608067454724

File: assets/urdf/xarm6/xarm6_1305_g2_movable_visual.urdf (robot description, URDF)
Before this commit: robot xarm6_1305_g2_movable_visual, 17 links, 16 joints
Joints:
- joint drive_joint: limit lower=0 upper=0.85 effort=50 velocity=2 -> lower=0.057210812728026743 upper=0.86509464599328212 effort=50 velocity=2.608067454724
- joint left_finger_joint: limit lower=0 upper=0.85 effort=50 velocity=2 -> lower=0.057210812728026743 upper=0.86509464599328212 effort=50 velocity=2.608067454724
- joint left_inner_knuckle_joint: limit lower=0 upper=0.85 effort=50 velocity=2 -> lower=0.057210812728026743 upper=0.86509464599328212 effort=50 velocity=2.608067454724
- joint right_finger_joint: limit lower=0 upper=0.85 effort=50 velocity=2 -> lower=0.057210812728026743 upper=0.86509464599328212 effort=50 velocity=2.608067454724
- joint right_inner_knuckle_joint: limit lower=0 upper=0.85 effort=50 velocity=2 -> lower=0.057210812728026743 upper=0.86509464599328212 effort=50 velocity=2.608067454724
- joint right_outer_knuckle_joint: limit lower=0 upper=0.85 effort=50 velocity=2 -> lower=0.057210812728026743 upper=0.86509464599328212 effort=50 velocity=2.608067454724

File: assets/urdf/xarm6/xarm6_1305_g2_visual.urdf (robot description, URDF)
Before this commit: robot xarm6_1305_g2_visual, 18 links, 17 joints
Joints:
- joint drive_joint: limit lower=0 upper=0.85 effort=50 velocity=2 -> lower=0.057210812728026743 upper=0.86509464599328212 effort=50 velocity=2.608067454724
- joint left_finger_joint: limit lower=0 upper=0.85 effort=50 velocity=2 -> lower=0.057210812728026743 upper=0.86509464599328212 effort=50 velocity=2.608067454724
- joint left_inner_knuckle_joint: limit lower=0 upper=0.85 effort=50 velocity=2 -> lower=0.057210812728026743 upper=0.86509464599328212 effort=50 velocity=2.608067454724
- joint right_finger_joint: limit lower=0 upper=0.85 effort=50 velocity=2 -> lower=0.057210812728026743 upper=0.86509464599328212 effort=50 velocity=2.608067454724
- joint right_inner_knuckle_joint: limit lower=0 upper=0.85 effort=50 velocity=2 -> lower=0.057210812728026743 upper=0.86509464599328212 effort=50 velocity=2.608067454724
- joint right_outer_knuckle_joint: limit lower=0 upper=0.85 effort=50 velocity=2 -> lower=0.057210812728026743 upper=0.86509464599328212 effort=50 velocity=2.608067454724

File: assets/urdf/xarm6/xarm6_with_gripper.urdf (robot description, URDF)
Before this commit: robot xarm6_with_gripper, 17 links, 16 joints
Joints:
- joint drive_joint: limit lower=0 upper=0.85 effort=50 velocity=2 -> lower=0.057210812728026743 upper=0.86509464599328212 effort=50 velocity=2.608067454724
- joint left_finger_joint: limit lower=0 upper=0.85 effort=50 velocity=2 -> lower=0.057210812728026743 upper=0.86509464599328212 effort=50 velocity=2.608067454724
- joint left_inner_knuckle_joint: limit lower=0 upper=0.85 effort=50 velocity=2 -> lower=0.057210812728026743 upper=0.86509464599328212 effort=50 velocity=2.608067454724
- joint right_finger_joint: limit lower=0 upper=0.85 effort=50 velocity=2 -> lower=0.057210812728026743 upper=0.86509464599328212 effort=50 velocity=2.608067454724
- joint right_inner_knuckle_joint: limit lower=0 upper=0.85 effort=50 velocity=2 -> lower=0.057210812728026743 upper=0.86509464599328212 effort=50 velocity=2.608067454724
- joint right_outer_knuckle_joint: limit lower=0 upper=0.85 effort=50 velocity=2 -> lower=0.057210812728026743 upper=0.86509464599328212 effort=50 velocity=2.608067454724

File: assets/urdf/xarm7/xarm7_1305_g2_movable_visual.urdf (robot description, URDF)
Before this commit: robot xarm7_1305_g2_movable_visual, 17 links, 16 joints
Joints:
- joint drive_joint: limit lower=0 upper=0.85 effort=50 velocity=2 -> lower=0.057210812728026743 upper=0.86509464599328212 effort=50 velocity=2.608067454724
- joint left_finger_joint: limit lower=0 upper=0.85 effort=50 velocity=2 -> lower=0.057210812728026743 upper=0.86509464599328212 effort=50 velocity=2.608067454724
- joint left_inner_knuckle_joint: limit lower=0 upper=0.85 effort=50 velocity=2 -> lower=0.057210812728026743 upper=0.86509464599328212 effort=50 velocity=2.608067454724
- joint right_finger_joint: limit lower=0 upper=0.85 effort=50 velocity=2 -> lower=0.057210812728026743 upper=0.86509464599328212 effort=50 velocity=2.608067454724
- joint right_inner_knuckle_joint: limit lower=0 upper=0.85 effort=50 velocity=2 -> lower=0.057210812728026743 upper=0.86509464599328212 effort=50 velocity=2.608067454724
- joint right_outer_knuckle_joint: limit lower=0 upper=0.85 effort=50 velocity=2 -> lower=0.057210812728026743 upper=0.86509464599328212 effort=50 velocity=2.608067454724

File: assets/urdf/xarm7/xarm7_1305_g2_visual.urdf (robot description, URDF)
Before this commit: robot xarm7_1305_g2_visual, 18 links, 17 joints
Joints:
- joint drive_joint: limit lower=0 upper=0.85 effort=50 velocity=2 -> lower=0.057210812728026743 upper=0.86509464599328212 effort=50 velocity=2.608067454724
- joint left_finger_joint: limit lower=0 upper=0.85 effort=50 velocity=2 -> lower=0.057210812728026743 upper=0.86509464599328212 effort=50 velocity=2.608067454724
- joint left_inner_knuckle_joint: limit lower=0 upper=0.85 effort=50 velocity=2 -> lower=0.057210812728026743 upper=0.86509464599328212 effort=50 velocity=2.608067454724
- joint right_finger_joint: limit lower=0 upper=0.85 effort=50 velocity=2 -> lower=0.057210812728026743 upper=0.86509464599328212 effort=50 velocity=2.608067454724
- joint right_inner_knuckle_joint: limit lower=0 upper=0.85 effort=50 velocity=2 -> lower=0.057210812728026743 upper=0.86509464599328212 effort=50 velocity=2.608067454724
- joint right_outer_knuckle_joint: limit lower=0 upper=0.85 effort=50 velocity=2 -> lower=0.057210812728026743 upper=0.86509464599328212 effort=50 velocity=2.608067454724
