Commit message: Release v0.1.1: Fix Bio Gripper G2 orientation and rename bio_gripper to bio_gripper_g2
- Fix Bio Gripper G2 flange orientation when mounted on arm (link5/link6/link7)
- Rename bio_gripper to bio_gripper_g2 across all assets, URDFs, examples, scripts
- Add missing with_bio_gripper_g2 parameter to xarm6_1305_visual_glb_urdf()
- Fix README --gripper-demo flag table to include Bio Gripper G2
- Move diagnostic/capture scripts and lerobot code to gitignored dev/
- Clean up stale bio_gripper files from git tracking
- Bump version 0.1.0 -> 0.1.1

Co-Authored-By: Claude <noreply@anthropic.com>

File: assets/urdf/gripper_g2/gripper_g2_movable_visual.urdf (robot description, URDF)
Before this commit: robot gripper_g2_movable_visual, 9 links, 8 joints
Links:
- link left_finger: geometry collision mesh filename=../gripper_g2/meshes/collision/left_finger.stl; visual mesh filename=../gripper_g2/meshes/visual/visual_glb/left_finger.glb
- link left_inner_knuckle: geometry collision mesh filename=../gripper_g2/meshes/collision/left_inner_knuckle.stl; visual mesh filename=../gripper_g2/meshes/visual/visual_glb/left_inner_knuckle.g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
- link left_outer_knuckle: geometry collision mesh filename=../gripper_g2/meshes/collision/left_outer_knuckle.stl; visual mesh filename=../gripper_g2/meshes/visual/visual_glb/left_outer_knuckle.g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
- link right_finger: geometry collision mesh filename=../gripper_g2/meshes/collision/right_finger.stl; visual mesh filename=../gripper_g2/meshes/visual/visual_glb/right_finger.glb
- link right_inner_knuckle: geometry collision mesh filename=../gripper_g2/meshes/collision/right_inner_knuckle.stl; visual mesh filename=../gripper_g2/meshes/visual/visual_glb/right_inner_knuckle.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
- link right_outer_knuckle: geometry collision mesh filename=../gripper_g2/meshes/collision/right_outer_knuckle.stl; visual mesh filename=../gripper_g2/meshes/visual/visual_glb/right_outer_knuckle.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
- link xarm_gripper_base_link: geometry collision mesh filename=../gripper_g2/meshes/collision/base_link.stl; visual mesh filename=../gripper_g2/meshes/visual/visual_glb/link6/base.glb

File: assets/urdf/uf850/uf850_g2_movable_visual.urdf (robot description, URDF)
Before this commit: robot uf850_g2_movable_visual, 16 links, 15 joints
Links:
- link left_finger: geometry collision mesh filename=../gripper_g2/meshes/collision/left_finger.stl; visual mesh filename=../gripper_g2/meshes/visual/visual_glb/left_finger.glb
- link left_inner_knuckle: geometry collision mesh filename=../gripper_g2/meshes/collision/left_inner_knuckle.stl; visual mesh filename=../gripper_g2/meshes/visual/visual_glb/left_inner_knuckle.g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
- link left_outer_knuckle: geometry collision mesh filename=../gripper_g2/meshes/collision/left_outer_knuckle.stl; visual mesh filename=../gripper_g2/meshes/visual/visual_glb/left_outer_knuckle.g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
- link right_finger: geometry collision mesh filename=../gripper_g2/meshes/collision/right_finger.stl; visual mesh filename=../gripper_g2/meshes/visual/visual_glb/right_finger.glb
- link right_inner_knuckle: geometry collision mesh filename=../gripper_g2/meshes/collision/right_inner_knuckle.stl; visual mesh filename=../gripper_g2/meshes/visual/visual_glb/right_inner_knuckle.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
- link right_outer_knuckle: geometry collision mesh filename=../gripper_g2/meshes/collision/right_outer_knuckle.stl; visual mesh filename=../gripper_g2/meshes/visual/visual_glb/right_outer_knuckle.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
- link xarm_gripper_base_link: geometry collision mesh filename=../gripper_g2/meshes/collision/base_link.stl; visual mesh filename=../gripper_g2/meshes/visual/visual_glb/link6/base.glb

File: assets/urdf/uf850/uf850_g2_visual.urdf (robot description, URDF)
Before this commit: robot uf850_g2_visual, 17 links, 16 joints
Links:
- link left_finger: geometry collision mesh filename=../gripper_g2/meshes/collision/left_finger.stl
- link left_inner_knuckle: geometry collision mesh filename=../gripper_g2/meshes/collision/left_inner_knuckle.stl
- link left_outer_knuckle: geometry collision mesh filename=../gripper_g2/meshes/collision/left_outer_knuckle.stl
- link right_finger: geometry collision mesh filename=../gripper_g2/meshes/collision/right_finger.stl
- link right_inner_knuckle: geometry collision mesh filename=../gripper_g2/meshes/collision/right_inner_knuckle.stl
- link right_outer_knuckle: geometry collision mesh filename=../gripper_g2/meshes/collision/right_outer_knuckle.stl
- link xarm_gripper_base_link: geometry collision mesh filename=../gripper_g2/meshes/collision/base_link.stl

File: assets/urdf/xarm5/xarm5_1305_g2_movable_visual.urdf (robot description, URDF)
Before this commit: robot xarm5_1305_g2_movable_visual, 15 links, 14 joints
Links:
- link left_finger: geometry collision mesh filename=../gripper_g2/meshes/collision/left_finger.stl; visual mesh filename=../gripper_g2/meshes/visual/visual_glb/left_finger.glb
- link left_inner_knuckle: geometry collision mesh filename=../gripper_g2/meshes/collision/left_inner_knuckle.stl; visual mesh filename=../gripper_g2/meshes/visual/visual_glb/left_inner_knuckle.g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
- link left_outer_knuckle: geometry collision mesh filename=../gripper_g2/meshes/collision/left_outer_knuckle.stl; visual mesh filename=../gripper_g2/meshes/visual/visual_glb/left_outer_knuckle.g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
- link right_finger: geometry collision mesh filename=../gripper_g2/meshes/collision/right_finger.stl; visual mesh filename=../gripper_g2/meshes/visual/visual_glb/right_finger.glb
- link right_inner_knuckle: geometry collision mesh filename=../gripper_g2/meshes/collision/right_inner_knuckle.stl; visual mesh filename=../gripper_g2/meshes/visual/visual_glb/right_inner_knuckle.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
- link right_outer_knuckle: geometry collision mesh filename=../gripper_g2/meshes/collision/right_outer_knuckle.stl; visual mesh filename=../gripper_g2/meshes/visual/visual_glb/right_outer_knuckle.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
- link xarm_gripper_base_link: geometry collision mesh filename=../gripper_g2/meshes/collision/base_link.stl; visual mesh filename=../gripper_g2/meshes/visual/visual_glb/link5/base.glb

File: assets/urdf/xarm5/xarm5_1305_g2_visual.urdf (robot description, URDF)
Before this commit: robot xarm5_1305_g2_visual, 16 links, 15 joints
Links:
- link left_finger: geometry collision mesh filename=../gripper_g2/meshes/collision/left_finger.stl
- link left_inner_knuckle: geometry collision mesh filename=../gripper_g2/meshes/collision/left_inner_knuckle.stl
- link left_outer_knuckle: geometry collision mesh filename=../gripper_g2/meshes/collision/left_outer_knuckle.stl
- link right_finger: geometry collision mesh filename=../gripper_g2/meshes/collision/right_finger.stl
- link right_inner_knuckle: geometry collision mesh filename=../gripper_g2/meshes/collision/right_inner_knuckle.stl
- link right_outer_knuckle: geometry collision mesh filename=../gripper_g2/meshes/collision/right_outer_knuckle.stl
- link xarm_gripper_base_link: geometry collision mesh filename=../gripper_g2/meshes/collision/base_link.stl

File: assets/urdf/xarm6/xarm6_1305_g2_movable_visual.urdf (robot description, URDF)
Before this commit: robot xarm6_1305_g2_movable_visual, 17 links, 16 joints
Links:
- link left_finger: geometry collision mesh filename=../gripper_g2/meshes/collision/left_finger.stl; visual mesh filename=../gripper_g2/meshes/visual/visual_glb/left_finger.glb
- link left_inner_knuckle: geometry collision mesh filename=../gripper_g2/meshes/collision/left_inner_knuckle.stl; visual mesh filename=../gripper_g2/meshes/visual/visual_glb/left_inner_knuckle.g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
- link left_outer_knuckle: geometry collision mesh filename=../gripper_g2/meshes/collision/left_outer_knuckle.stl; visual mesh filename=../gripper_g2/meshes/visual/visual_glb/left_outer_knuckle.g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
- link right_finger: geometry collision mesh filename=../gripper_g2/meshes/collision/right_finger.stl; visual mesh filename=../gripper_g2/meshes/visual/visual_glb/right_finger.glb
- link right_inner_knuckle: geometry collision mesh filename=../gripper_g2/meshes/collision/right_inner_knuckle.stl; visual mesh filename=../gripper_g2/meshes/visual/visual_glb/right_inner_knuckle.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
- link right_outer_knuckle: geometry collision mesh filename=../gripper_g2/meshes/collision/right_outer_knuckle.stl; visual mesh filename=../gripper_g2/meshes/visual/visual_glb/right_outer_knuckle.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
- link xarm_gripper_base_link: geometry collision mesh filename=../gripper_g2/meshes/collision/base_link.stl; visual mesh filename=../gripper_g2/meshes/visual/visual_glb/link6/base.glb

File: assets/urdf/xarm6/xarm6_1305_g2_visual.urdf (robot description, URDF)
Before this commit: robot xarm6_1305_g2_visual, 18 links, 17 joints
Links:
- link left_finger: geometry collision mesh filename=../gripper_g2/meshes/collision/left_finger.stl
- link left_inner_knuckle: geometry collision mesh filename=../gripper_g2/meshes/collision/left_inner_knuckle.stl
- link left_outer_knuckle: geometry collision mesh filename=../gripper_g2/meshes/collision/left_outer_knuckle.stl
- link right_finger: geometry collision mesh filename=../gripper_g2/meshes/collision/right_finger.stl
- link right_inner_knuckle: geometry collision mesh filename=../gripper_g2/meshes/collision/right_inner_knuckle.stl
- link right_outer_knuckle: geometry collision mesh filename=../gripper_g2/meshes/collision/right_outer_knuckle.stl
- link xarm_gripper_base_link: geometry collision mesh filename=../gripper_g2/meshes/collision/base_link.stl

File: assets/urdf/xarm6/xarm6_with_gripper.urdf (robot description, URDF)
Before this commit: robot xarm6_with_gripper, 17 links, 16 joints
Links:
- link left_finger: geometry collision mesh filename=../gripper_g2/meshes/collision/left_finger.stl; visual mesh filename=../gripper_g2/meshes/collision/left_finger.stl
- link left_inner_knuckle: geometry collision mesh filename=../gripper_g2/meshes/collision/left_inner_knuckle.stl; visual mesh filename=../gripper_g2/meshes/collision/left_inner_knuckle.stl
- link left_outer_knuckle: geometry collision mesh filename=../gripper_g2/meshes/collision/left_outer_knuckle.stl; visual mesh filename=../gripper_g2/meshes/collision/left_outer_knuckle.stl
- link right_finger: geometry collision mesh filename=../gripper_g2/meshes/collision/right_finger.stl; visual mesh filename=../gripper_g2/meshes/collision/right_finger.stl
- link right_inner_knuckle: geometry collision mesh filename=../gripper_g2/meshes/collision/right_inner_knuckle.stl; visual mesh filename=../gripper_g2/meshes/collision/right_inner_knuckle.stl
- link right_outer_knuckle: geometry collision mesh filename=../gripper_g2/meshes/collision/right_outer_knuckle.stl; visual mesh filename=../gripper_g2/meshes/collision/right_outer_knuckle.stl
- link xarm_gripper_base_link: geometry collision mesh filename=../gripper_g2/meshes/collision/base_link.stl; visual mesh filename=../gripper_g2/meshes/collision/base_link.stl

File: assets/urdf/xarm7/xarm7_1305_g2_movable_visual.urdf (robot description, URDF)
Before this commit: robot xarm7_1305_g2_movable_visual, 17 links, 16 joints
Links:
- link left_finger: geometry collision mesh filename=../gripper_g2/meshes/collision/left_finger.stl; visual mesh filename=../gripper_g2/meshes/visual/visual_glb/left_finger.glb
- link left_inner_knuckle: geometry collision mesh filename=../gripper_g2/meshes/collision/left_inner_knuckle.stl; visual mesh filename=../gripper_g2/meshes/visual/visual_glb/left_inner_knuckle.g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
- link left_outer_knuckle: geometry collision mesh filename=../gripper_g2/meshes/collision/left_outer_knuckle.stl; visual mesh filename=../gripper_g2/meshes/visual/visual_glb/left_outer_knuckle.g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
- link right_finger: geometry collision mesh filename=../gripper_g2/meshes/collision/right_finger.stl; visual mesh filename=../gripper_g2/meshes/visual/visual_glb/right_finger.glb
- link right_inner_knuckle: geometry collision mesh filename=../gripper_g2/meshes/collision/right_inner_knuckle.stl; visual mesh filename=../gripper_g2/meshes/visual/visual_glb/right_inner_knuckle.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
- link right_outer_knuckle: geometry collision mesh filename=../gripper_g2/meshes/collision/right_outer_knuckle.stl; visual mesh filename=../gripper_g2/meshes/visual/visual_glb/right_outer_knuckle.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
- link xarm_gripper_base_link: geometry collision mesh filename=../gripper_g2/meshes/collision/base_link.stl; visual mesh filename=../gripper_g2/meshes/visual/visual_glb/link7/base.glb

File: assets/urdf/xarm7/xarm7_1305_g2_visual.urdf (robot description, URDF)
Before this commit: robot xarm7_1305_g2_visual, 18 links, 17 joints
Links:
- link left_finger: geometry collision mesh filename=../gripper_g2/meshes/collision/left_finger.stl
- link left_inner_knuckle: geometry collision mesh filename=../gripper_g2/meshes/collision/left_inner_knuckle.stl
- link left_outer_knuckle: geometry collision mesh filename=../gripper_g2/meshes/collision/left_outer_knuckle.stl
- link right_finger: geometry collision mesh filename=../gripper_g2/meshes/collision/right_finger.stl
- link right_inner_knuckle: geometry collision mesh filename=../gripper_g2/meshes/collision/right_inner_knuckle.stl
- link right_outer_knuckle: geometry collision mesh filename=../gripper_g2/meshes/collision/right_outer_knuckle.stl
- link xarm_gripper_base_link: geometry collision mesh filename=../gripper_g2/meshes/collision/base_link.stl
