Commit message: Release 0.1.3: Genesis 1.2.0 and Bio G2 xArm7 flange fix.
Raise minimum genesis-world to 1.2.0 (refresh_rate API) and fix link7 pin-hole mirroring that sank Bio Gripper G2 into the arm flange.

Co-authored-by: Cursor <cursoragent@cursor.com>

File: assets/urdf/uf850/uf850_bio_gripper_g2_movable_visual.glb.urdf (robot description, URDF)
Before this commit: robot uf850_bio_gripper_g2_movable_visual.glb, 12 links, 11 joints
Joints:
- joint bio_gripper_g2_attach: origin xyz=0.034285 0.000413 -0.001674 rpy=0.00018025 0.01490249 -0.00018304 -> xyz=0.034255 0.000449 -0.001869 rpy=0.00040363 0.01305476 -0.00292163

Commit message: Release v0.1.4: Bio Gripper G2 flange mount offset fix.
Move static Bio G2 GLB to canonical gripper base frame and eliminate
hardcoded Rx(pi) attach origins.  Both static and movable combo URDFs
now share relocalized per-profile attach origins from relocalize_metrics.
UF850 flange mounting offset reduced from ~12mm to ~3.5mm hole fit.

Co-Authored-By: Claude <noreply@anthropic.com>

File: assets/urdf/uf850/uf850_bio_gripper_g2_movable_visual.glb.urdf (robot description, URDF)
Before this commit: robot uf850_bio_gripper_g2_movable_visual.glb, 12 links, 11 joints
Joints:
- joint bio_gripper_g2_attach: origin xyz=0.034255 0.000449 -0.001869 rpy=0.00040363 0.01305476 -0.00292163 -> xyz=0.024657 0.012975 -0.000386 rpy=0.00000000 0.00000000 0.47492066

File: assets/urdf/uf850/uf850_bio_gripper_g2_visual.glb.urdf (robot description, URDF)
Before this commit: robot uf850_bio_gripper_g2_visual.glb, 13 links, 12 joints
Joints:
- joint bio_gripper_g2_attach: origin xyz=0 0 0 rpy=3.14159265 0 0 -> xyz=0.024657 0.012975 -0.000386 rpy=0.00000000 0.00000000 0.47492066
- joint bio_gripper_g2_visual_fix: origin xyz=0 0 0 rpy=3.14159265 0 0 -> xyz=0.024657 0.012975 -0.000386 rpy=0.00000000 0.00000000 0.47492066

File: assets/urdf/xarm5/xarm5_1305_bio_gripper_g2_movable_visual.glb.urdf (robot description, URDF)
Before this commit: robot xarm5_1305_bio_gripper_g2_movable_visual.glb, 11 links, 10 joints
Joints:
- joint bio_gripper_g2_attach: origin xyz=0.026044 -0.000488 -0.000697 rpy=0.00000000 0.00000000 0.00702875 -> xyz=0.026044 -0.000867 -0.000697 rpy=0.00000000 0.00000000 -0.00702875

File: assets/urdf/xarm5/xarm5_1305_bio_gripper_g2_visual.glb.urdf (robot description, URDF)
Before this commit: robot xarm5_1305_bio_gripper_g2_visual.glb, 12 links, 11 joints
Joints:
- joint bio_gripper_g2_attach: origin xyz=0 0 0 rpy=3.14159265 0 0 -> xyz=0.026044 -0.000867 -0.000697 rpy=0.00000000 0.00000000 -0.00702875
- joint bio_gripper_g2_visual_fix: origin xyz=0 0 0 rpy=3.14159265 0 0 -> xyz=0.026044 -0.000867 -0.000697 rpy=0.00000000 0.00000000 -0.00702875

File: assets/urdf/xarm6/xarm6_1305_bio_gripper_g2_movable_visual.glb.urdf (robot description, URDF)
Before this commit: robot xarm6_1305_bio_gripper_g2_movable_visual.glb, 13 links, 12 joints
Joints:
- joint bio_gripper_g2_attach: origin xyz=0.027018 -0.000335 -0.000692 rpy=0.00000000 0.00000000 0.00706128 -> xyz=0.027018 -0.000715 -0.000692 rpy=0.00000000 0.00000000 -0.00706128

File: assets/urdf/xarm6/xarm6_1305_bio_gripper_g2_visual.glb.urdf (robot description, URDF)
Before this commit: robot xarm6_1305_bio_gripper_g2_visual.glb, 14 links, 13 joints
Joints:
- joint bio_gripper_g2_attach: origin xyz=0 0 0 rpy=3.14159265 0 0 -> xyz=0.027018 -0.000715 -0.000692 rpy=0.00000000 0.00000000 -0.00706128
- joint bio_gripper_g2_visual_fix: origin xyz=0 0 0 rpy=3.14159265 0 0 -> xyz=0.027018 -0.000715 -0.000692 rpy=0.00000000 0.00000000 -0.00706128

File: assets/urdf/xarm7/xarm7_1305_bio_gripper_g2_movable_visual.glb.urdf (robot description, URDF)
Before this commit: robot xarm7_1305_bio_gripper_g2_movable_visual.glb, 13 links, 12 joints
Joints:
- joint bio_gripper_g2_attach: origin xyz=0.026931 -0.000459 -0.000760 rpy=0.00000000 0.00000000 0.00784664 -> xyz=0.026931 -0.000882 -0.000760 rpy=0.00000000 0.00000000 -0.00784664

File: assets/urdf/xarm7/xarm7_1305_bio_gripper_g2_visual.glb.urdf (robot description, URDF)
Before this commit: robot xarm7_1305_bio_gripper_g2_visual.glb, 14 links, 13 joints
Joints:
- joint bio_gripper_g2_attach: origin xyz=0 0 0 rpy=3.14159265 0 0 -> xyz=0.026931 -0.000882 -0.000760 rpy=0.00000000 0.00000000 -0.00784664
- joint bio_gripper_g2_visual_fix: origin xyz=0 0 0 rpy=3.14159265 0 0 -> xyz=0.026931 -0.000882 -0.000760 rpy=0.00000000 0.00000000 -0.00784664
