Commit message: Release v0.2.0: modular package layout and STL collision meshes.
Breaking refactor groups APIs by domain; xArm5/6/7 collision OBJ→STL;
five-robot dynamics validation with documented xArm5 pose4 Genesis limitation.

Co-authored-by: Cursor <cursoragent@cursor.com>

File: assets/urdf/xarm5/xarm5_1305.urdf (robot description, URDF)
Before this commit: robot gen, 7 links, 6 joints
Links:
- link link1: geometry collision mesh filename=meshes/xarm5_1305/collision/link1.stl; visual mesh filename=meshes/xarm5_1305/visual/link1.stl
- link link2: geometry collision mesh filename=meshes/xarm5_1305/collision/link2.stl; visual mesh filename=meshes/xarm5_1305/visual/link2.stl
- link link3: geometry collision mesh filename=meshes/xarm5_1305/collision/link3.stl; visual mesh filename=meshes/xarm5_1305/visual/link3.stl
- link link4: geometry collision mesh filename=meshes/xarm5_1305/collision/link4.stl; visual mesh filename=meshes/xarm5_1305/visual/link4.stl
- link link5: geometry collision mesh filename=meshes/xarm5_1305/collision/link5.stl; visual mesh filename=meshes/xarm5_1305/visual/link5.stl
- link link_base: geometry collision mesh filename=meshes/xarm5_1305/collision/link_base.stl; visual mesh filename=meshes/xarm5_1305/visual/link_base.stl

File: assets/urdf/xarm5/xarm5_1305_bio_gripper_g2_movable_visual.glb.urdf (robot description, URDF)
Before this commit: robot xarm5_1305_bio_gripper_g2_movable_visual.glb, 11 links, 10 joints
Links:
- link link1: geometry collision mesh filename=meshes/xarm5_1305/collision/link1.stl; visual mesh filename=meshes/xarm5_1305/visual_glb/link1.glb
- link link2: geometry collision mesh filename=meshes/xarm5_1305/collision/link2.stl; visual mesh filename=meshes/xarm5_1305/visual_glb/link2.glb
- link link3: geometry collision mesh filename=meshes/xarm5_1305/collision/link3.stl; visual mesh filename=meshes/xarm5_1305/visual_glb/link3.glb
- link link4: geometry collision mesh filename=meshes/xarm5_1305/collision/link4.stl; visual mesh filename=meshes/xarm5_1305/visual_glb/link4.glb
- link link5: geometry collision mesh filename=meshes/xarm5_1305/collision/link5.stl; visual mesh filename=meshes/xarm5_1305/visual_glb/link5.glb
- link link_base: geometry collision mesh filename=meshes/xarm5_1305/collision/link_base.stl; visual mesh filename=meshes/xarm5_1305/visual_glb/link_base.glb

File: assets/urdf/xarm5/xarm5_1305_bio_gripper_g2_visual.glb.urdf (robot description, URDF)
Before this commit: robot xarm5_1305_bio_gripper_g2_visual.glb, 12 links, 11 joints
Links:
- link link1: geometry collision mesh filename=meshes/xarm5_1305/collision/link1.stl; visual mesh filename=meshes/xarm5_1305/visual_glb/link1.glb
- link link2: geometry collision mesh filename=meshes/xarm5_1305/collision/link2.stl; visual mesh filename=meshes/xarm5_1305/visual_glb/link2.glb
- link link3: geometry collision mesh filename=meshes/xarm5_1305/collision/link3.stl; visual mesh filename=meshes/xarm5_1305/visual_glb/link3.glb
- link link4: geometry collision mesh filename=meshes/xarm5_1305/collision/link4.stl; visual mesh filename=meshes/xarm5_1305/visual_glb/link4.glb
- link link5: geometry collision mesh filename=meshes/xarm5_1305/collision/link5.stl; visual mesh filename=meshes/xarm5_1305/visual_glb/link5.glb
- link link_base: geometry collision mesh filename=meshes/xarm5_1305/collision/link_base.stl; visual mesh filename=meshes/xarm5_1305/visual_glb/link_base.glb

File: assets/urdf/xarm5/xarm5_1305_g2_movable_visual.urdf (robot description, URDF)
Before this commit: robot xarm5_1305_g2_movable_visual, 15 links, 14 joints
Links:
- link link1: geometry collision mesh filename=meshes/xarm5_1305/collision/link1.stl; visual mesh filename=meshes/xarm5_1305/visual_glb/link1.glb
- link link2: geometry collision mesh filename=meshes/xarm5_1305/collision/link2.stl; visual mesh filename=meshes/xarm5_1305/visual_glb/link2.glb
- link link3: geometry collision mesh filename=meshes/xarm5_1305/collision/link3.stl; visual mesh filename=meshes/xarm5_1305/visual_glb/link3.glb
- link link4: geometry collision mesh filename=meshes/xarm5_1305/collision/link4.stl; visual mesh filename=meshes/xarm5_1305/visual_glb/link4.glb
- link link5: geometry collision mesh filename=meshes/xarm5_1305/collision/link5.stl; visual mesh filename=meshes/xarm5_1305/visual_glb/link5.glb
- link link_base: geometry collision mesh filename=meshes/xarm5_1305/collision/link_base.stl; visual mesh filename=meshes/xarm5_1305/visual_glb/link_base.glb

File: assets/urdf/xarm5/xarm5_1305_g2_visual.urdf (robot description, URDF)
Before this commit: robot xarm5_1305_g2_visual, 16 links, 15 joints
Links:
- link link1: geometry collision mesh filename=meshes/xarm5_1305/collision/link1.stl; visual mesh filename=meshes/xarm5_1305/visual_glb/link1.glb
- link link2: geometry collision mesh filename=meshes/xarm5_1305/collision/link2.stl; visual mesh filename=meshes/xarm5_1305/visual_glb/link2.glb
- link link3: geometry collision mesh filename=meshes/xarm5_1305/collision/link3.stl; visual mesh filename=meshes/xarm5_1305/visual_glb/link3.glb
- link link4: geometry collision mesh filename=meshes/xarm5_1305/collision/link4.stl; visual mesh filename=meshes/xarm5_1305/visual_glb/link4.glb
- link link5: geometry collision mesh filename=meshes/xarm5_1305/collision/link5.stl; visual mesh filename=meshes/xarm5_1305/visual_glb/link5.glb
- link link_base: geometry collision mesh filename=meshes/xarm5_1305/collision/link_base.stl; visual mesh filename=meshes/xarm5_1305/visual_glb/link_base.glb

File: assets/urdf/xarm5/xarm5_1305_visual.glb.urdf (robot description, URDF)
Before this commit: robot gen, 7 links, 6 joints
Links:
- link link1: geometry collision mesh filename=meshes/xarm5_1305/collision/link1.stl; visual mesh filename=meshes/xarm5_1305/visual_glb/link1.glb
- link link2: geometry collision mesh filename=meshes/xarm5_1305/collision/link2.stl; visual mesh filename=meshes/xarm5_1305/visual_glb/link2.glb
- link link3: geometry collision mesh filename=meshes/xarm5_1305/collision/link3.stl; visual mesh filename=meshes/xarm5_1305/visual_glb/link3.glb
- link link4: geometry collision mesh filename=meshes/xarm5_1305/collision/link4.stl; visual mesh filename=meshes/xarm5_1305/visual_glb/link4.glb
- link link5: geometry collision mesh filename=meshes/xarm5_1305/collision/link5.stl; visual mesh filename=meshes/xarm5_1305/visual_glb/link5.glb
- link link_base: geometry collision mesh filename=meshes/xarm5_1305/collision/link_base.stl; visual mesh filename=meshes/xarm5_1305/visual_glb/link_base.glb

File: assets/urdf/xarm6/xarm6_1305.urdf (robot description, URDF)
Before this commit: robot xarm6_1305, 9 links, 8 joints
Links:
- link link1: geometry collision mesh filename=meshes/xarm6_1305/collision/link1.stl; visual mesh filename=meshes/xarm6_1305/visual/link1.stl
- link link2: geometry collision mesh filename=meshes/xarm6_1305/collision/link2.stl; visual mesh filename=meshes/xarm6_1305/visual/link2.stl
- link link3: geometry collision mesh filename=meshes/xarm6_1305/collision/link3.stl; visual mesh filename=meshes/xarm6_1305/visual/link3.stl
- link link4: geometry collision mesh filename=meshes/xarm6_1305/collision/link4.stl; visual mesh filename=meshes/xarm6_1305/visual/link4.stl
- link link5: geometry collision mesh filename=meshes/xarm6_1305/collision/link5.stl; visual mesh filename=meshes/xarm6_1305/visual/link5.stl
- link link6: geometry collision mesh filename=meshes/xarm6_1305/collision/link6.stl; visual mesh filename=meshes/xarm6_1305/visual/link6.stl
- link link_base: geometry collision mesh filename=meshes/xarm6_1305/collision/link_base.stl; visual mesh filename=meshes/xarm6_1305/visual/link_base.stl

File: assets/urdf/xarm6/xarm6_1305_bio_gripper_g2_movable_visual.glb.urdf (robot description, URDF)
Before this commit: robot xarm6_1305_bio_gripper_g2_movable_visual.glb, 13 links, 12 joints
Links:
- link link1: geometry collision mesh filename=meshes/xarm6_1305/collision/link1.stl; visual mesh filename=meshes/xarm6_1305/visual_glb/link1.glb
- link link2: geometry collision mesh filename=meshes/xarm6_1305/collision/link2.stl; visual mesh filename=meshes/xarm6_1305/visual_glb/link2.glb
- link link3: geometry collision mesh filename=meshes/xarm6_1305/collision/link3.stl; visual mesh filename=meshes/xarm6_1305/visual_glb/link3.glb
- link link4: geometry collision mesh filename=meshes/xarm6_1305/collision/link4.stl; visual mesh filename=meshes/xarm6_1305/visual_glb/link4.glb
- link link5: geometry collision mesh filename=meshes/xarm6_1305/collision/link5.stl; visual mesh filename=meshes/xarm6_1305/visual_glb/link5.glb
- link link6: geometry collision mesh filename=meshes/xarm6_1305/collision/link6.stl; visual mesh filename=meshes/xarm6_1305/visual_glb/link6.glb
- link link_base: geometry collision mesh filename=meshes/xarm6_1305/collision/link_base.stl; visual mesh filename=meshes/xarm6_1305/visual_glb/link_base.glb

File: assets/urdf/xarm6/xarm6_1305_bio_gripper_g2_visual.glb.urdf (robot description, URDF)
Before this commit: robot xarm6_1305_bio_gripper_g2_visual.glb, 14 links, 13 joints
Links:
- link link1: geometry collision mesh filename=meshes/xarm6_1305/collision/link1.stl; visual mesh filename=meshes/xarm6_1305/visual_glb/link1.glb
- link link2: geometry collision mesh filename=meshes/xarm6_1305/collision/link2.stl; visual mesh filename=meshes/xarm6_1305/visual_glb/link2.glb
- link link3: geometry collision mesh filename=meshes/xarm6_1305/collision/link3.stl; visual mesh filename=meshes/xarm6_1305/visual_glb/link3.glb
- link link4: geometry collision mesh filename=meshes/xarm6_1305/collision/link4.stl; visual mesh filename=meshes/xarm6_1305/visual_glb/link4.glb
- link link5: geometry collision mesh filename=meshes/xarm6_1305/collision/link5.stl; visual mesh filename=meshes/xarm6_1305/visual_glb/link5.glb
- link link6: geometry collision mesh filename=meshes/xarm6_1305/collision/link6.stl; visual mesh filename=meshes/xarm6_1305/visual_glb/link6.glb
- link link_base: geometry collision mesh filename=meshes/xarm6_1305/collision/link_base.stl; visual mesh filename=meshes/xarm6_1305/visual_glb/link_base.glb

File: assets/urdf/xarm6/xarm6_1305_g2_movable_visual.urdf (robot description, URDF)
Before this commit: robot xarm6_1305_g2_movable_visual, 17 links, 16 joints
Links:
- link link1: geometry collision mesh filename=meshes/xarm6_1305/collision/link1.stl; visual mesh filename=meshes/xarm6_1305/visual_glb/link1.glb
- link link2: geometry collision mesh filename=meshes/xarm6_1305/collision/link2.stl; visual mesh filename=meshes/xarm6_1305/visual_glb/link2.glb
- link link3: geometry collision mesh filename=meshes/xarm6_1305/collision/link3.stl; visual mesh filename=meshes/xarm6_1305/visual_glb/link3.glb
- link link4: geometry collision mesh filename=meshes/xarm6_1305/collision/link4.stl; visual mesh filename=meshes/xarm6_1305/visual_glb/link4.glb
- link link5: geometry collision mesh filename=meshes/xarm6_1305/collision/link5.stl; visual mesh filename=meshes/xarm6_1305/visual_glb/link5.glb
- link link6: geometry collision mesh filename=meshes/xarm6_1305/collision/link6.stl; visual mesh filename=meshes/xarm6_1305/visual_glb/link6.glb
- link link_base: geometry collision mesh filename=meshes/xarm6_1305/collision/link_base.stl; visual mesh filename=meshes/xarm6_1305/visual_glb/link_base.glb

File: assets/urdf/xarm6/xarm6_1305_g2_visual.urdf (robot description, URDF)
Before this commit: robot xarm6_1305_g2_visual, 18 links, 17 joints
Links:
- link link1: geometry collision mesh filename=meshes/xarm6_1305/collision/link1.stl; visual mesh filename=meshes/xarm6_1305/visual_glb/link1.glb
- link link2: geometry collision mesh filename=meshes/xarm6_1305/collision/link2.stl; visual mesh filename=meshes/xarm6_1305/visual_glb/link2.glb
- link link3: geometry collision mesh filename=meshes/xarm6_1305/collision/link3.stl; visual mesh filename=meshes/xarm6_1305/visual_glb/link3.glb
- link link4: geometry collision mesh filename=meshes/xarm6_1305/collision/link4.stl; visual mesh filename=meshes/xarm6_1305/visual_glb/link4.glb
- link link5: geometry collision mesh filename=meshes/xarm6_1305/collision/link5.stl; visual mesh filename=meshes/xarm6_1305/visual_glb/link5.glb
- link link6: geometry collision mesh filename=meshes/xarm6_1305/collision/link6.stl; visual mesh filename=meshes/xarm6_1305/visual_glb/link6.glb
- link link_base: geometry collision mesh filename=meshes/xarm6_1305/collision/link_base.stl; visual mesh filename=meshes/xarm6_1305/visual_glb/link_base.glb

File: assets/urdf/xarm6/xarm6_1305_visual.glb.urdf (robot description, URDF)
Before this commit: robot xarm6_1305_visual_glb, 9 links, 8 joints
Links:
- link link1: geometry collision mesh filename=meshes/xarm6_1305/collision/link1.stl; visual mesh filename=meshes/xarm6_1305/visual_glb/link1.glb
- link link2: geometry collision mesh filename=meshes/xarm6_1305/collision/link2.stl; visual mesh filename=meshes/xarm6_1305/visual_glb/link2.glb
- link link3: geometry collision mesh filename=meshes/xarm6_1305/collision/link3.stl; visual mesh filename=meshes/xarm6_1305/visual_glb/link3.glb
- link link4: geometry collision mesh filename=meshes/xarm6_1305/collision/link4.stl; visual mesh filename=meshes/xarm6_1305/visual_glb/link4.glb
- link link5: geometry collision mesh filename=meshes/xarm6_1305/collision/link5.stl; visual mesh filename=meshes/xarm6_1305/visual_glb/link5.glb
- link link6: geometry collision mesh filename=meshes/xarm6_1305/collision/link6.stl; visual mesh filename=meshes/xarm6_1305/visual_glb/link6.glb
- link link_base: geometry collision mesh filename=meshes/xarm6_1305/collision/link_base.stl; visual mesh filename=meshes/xarm6_1305/visual_glb/link_base.glb

File: assets/urdf/xarm6/xarm6_with_gripper.urdf (robot description, URDF)
Before this commit: robot xarm6_with_gripper, 17 links, 16 joints
Links:
- link link1: geometry collision mesh filename=meshes/xarm6_1305/collision/link1.stl; visual mesh filename=meshes/xarm6_1305/visual/link1.stl
- link link2: geometry collision mesh filename=meshes/xarm6_1305/collision/link2.stl; visual mesh filename=meshes/xarm6_1305/visual/link2.stl
- link link3: geometry collision mesh filename=meshes/xarm6_1305/collision/link3.stl; visual mesh filename=meshes/xarm6_1305/visual/link3.stl
- link link4: geometry collision mesh filename=meshes/xarm6_1305/collision/link4.stl; visual mesh filename=meshes/xarm6_1305/visual/link4.stl
- link link5: geometry collision mesh filename=meshes/xarm6_1305/collision/link5.stl; visual mesh filename=meshes/xarm6_1305/visual/link5.stl
- link link6: geometry collision mesh filename=meshes/xarm6_1305/collision/link6.stl; visual mesh filename=meshes/xarm6_1305/visual/link6.stl
- link link_base: geometry collision mesh filename=meshes/xarm6_1305/collision/link_base.stl; visual mesh filename=meshes/xarm6_1305/visual/link_base.stl

File: assets/urdf/xarm7/xarm7_1305.urdf (robot description, URDF)
Before this commit: robot gen, 9 links, 8 joints
Links:
- link link1: geometry collision mesh filename=meshes/xarm7_1305/collision/link1.stl; visual mesh filename=meshes/xarm7_1305/visual/link1.stl
- link link2: geometry collision mesh filename=meshes/xarm7_1305/collision/link2.stl; visual mesh filename=meshes/xarm7_1305/visual/link2.stl
- link link3: geometry collision mesh filename=meshes/xarm7_1305/collision/link3.stl; visual mesh filename=meshes/xarm7_1305/visual/link3.stl
- link link4: geometry collision mesh filename=meshes/xarm7_1305/collision/link4.stl; visual mesh filename=meshes/xarm7_1305/visual/link4.stl
- link link5: geometry collision mesh filename=meshes/xarm7_1305/collision/link5.stl; visual mesh filename=meshes/xarm7_1305/visual/link5.stl
- link link6: geometry collision mesh filename=meshes/xarm7_1305/collision/link6.stl; visual mesh filename=meshes/xarm7_1305/visual/link6.stl
- link link7: geometry collision mesh filename=meshes/xarm7_1305/collision/link7.stl; visual mesh filename=meshes/xarm7_1305/visual/link7.stl
- link link_base: geometry collision mesh filename=meshes/xarm7_1305/collision/link_base.stl; visual mesh filename=meshes/xarm7_1305/visual/link_base.stl

File: assets/urdf/xarm7/xarm7_1305_bio_gripper_g2_movable_visual.glb.urdf (robot description, URDF)
Before this commit: robot xarm7_1305_bio_gripper_g2_movable_visual.glb, 13 links, 12 joints
Links:
- link link1: geometry collision mesh filename=meshes/xarm7_1305/collision/link1.stl; visual mesh filename=meshes/xarm7_1305/visual_glb/link1.glb
- link link2: geometry collision mesh filename=meshes/xarm7_1305/collision/link2.stl; visual mesh filename=meshes/xarm7_1305/visual_glb/link2.glb
- link link3: geometry collision mesh filename=meshes/xarm7_1305/collision/link3.stl; visual mesh filename=meshes/xarm7_1305/visual_glb/link3.glb
- link link4: geometry collision mesh filename=meshes/xarm7_1305/collision/link4.stl; visual mesh filename=meshes/xarm7_1305/visual_glb/link4.glb
- link link5: geometry collision mesh filename=meshes/xarm7_1305/collision/link5.stl; visual mesh filename=meshes/xarm7_1305/visual_glb/link5.glb
- link link6: geometry collision mesh filename=meshes/xarm7_1305/collision/link6.stl; visual mesh filename=meshes/xarm7_1305/visual_glb/link6.glb
- link link7: geometry collision mesh filename=meshes/xarm7_1305/collision/link7.stl; visual mesh filename=meshes/xarm7_1305/visual_glb/link7.glb
- link link_base: geometry collision mesh filename=meshes/xarm7_1305/collision/link_base.stl; visual mesh filename=meshes/xarm7_1305/visual_glb/link_base.glb

File: assets/urdf/xarm7/xarm7_1305_bio_gripper_g2_visual.glb.urdf (robot description, URDF)
Before this commit: robot xarm7_1305_bio_gripper_g2_visual.glb, 14 links, 13 joints
Links:
- link link1: geometry collision mesh filename=meshes/xarm7_1305/collision/link1.stl; visual mesh filename=meshes/xarm7_1305/visual_glb/link1.glb
- link link2: geometry collision mesh filename=meshes/xarm7_1305/collision/link2.stl; visual mesh filename=meshes/xarm7_1305/visual_glb/link2.glb
- link link3: geometry collision mesh filename=meshes/xarm7_1305/collision/link3.stl; visual mesh filename=meshes/xarm7_1305/visual_glb/link3.glb
- link link4: geometry collision mesh filename=meshes/xarm7_1305/collision/link4.stl; visual mesh filename=meshes/xarm7_1305/visual_glb/link4.glb
- link link5: geometry collision mesh filename=meshes/xarm7_1305/collision/link5.stl; visual mesh filename=meshes/xarm7_1305/visual_glb/link5.glb
- link link6: geometry collision mesh filename=meshes/xarm7_1305/collision/link6.stl; visual mesh filename=meshes/xarm7_1305/visual_glb/link6.glb
- link link7: geometry collision mesh filename=meshes/xarm7_1305/collision/link7.stl; visual mesh filename=meshes/xarm7_1305/visual_glb/link7.glb
- link link_base: geometry collision mesh filename=meshes/xarm7_1305/collision/link_base.stl; visual mesh filename=meshes/xarm7_1305/visual_glb/link_base.glb

File: assets/urdf/xarm7/xarm7_1305_g2_movable_visual.urdf (robot description, URDF)
Before this commit: robot xarm7_1305_g2_movable_visual, 17 links, 16 joints
Links:
- link link1: geometry collision mesh filename=meshes/xarm7_1305/collision/link1.stl; visual mesh filename=meshes/xarm7_1305/visual_glb/link1.glb
- link link2: geometry collision mesh filename=meshes/xarm7_1305/collision/link2.stl; visual mesh filename=meshes/xarm7_1305/visual_glb/link2.glb
- link link3: geometry collision mesh filename=meshes/xarm7_1305/collision/link3.stl; visual mesh filename=meshes/xarm7_1305/visual_glb/link3.glb
- link link4: geometry collision mesh filename=meshes/xarm7_1305/collision/link4.stl; visual mesh filename=meshes/xarm7_1305/visual_glb/link4.glb
- link link5: geometry collision mesh filename=meshes/xarm7_1305/collision/link5.stl; visual mesh filename=meshes/xarm7_1305/visual_glb/link5.glb
- link link6: geometry collision mesh filename=meshes/xarm7_1305/collision/link6.stl; visual mesh filename=meshes/xarm7_1305/visual_glb/link6.glb
- link link7: geometry collision mesh filename=meshes/xarm7_1305/collision/link7.stl; visual mesh filename=meshes/xarm7_1305/visual_glb/link7.glb
- link link_base: geometry collision mesh filename=meshes/xarm7_1305/collision/link_base.stl; visual mesh filename=meshes/xarm7_1305/visual_glb/link_base.glb

File: assets/urdf/xarm7/xarm7_1305_g2_visual.urdf (robot description, URDF)
Before this commit: robot xarm7_1305_g2_visual, 18 links, 17 joints
Links:
- link link1: geometry collision mesh filename=meshes/xarm7_1305/collision/link1.stl; visual mesh filename=meshes/xarm7_1305/visual_glb/link1.glb
- link link2: geometry collision mesh filename=meshes/xarm7_1305/collision/link2.stl; visual mesh filename=meshes/xarm7_1305/visual_glb/link2.glb
- link link3: geometry collision mesh filename=meshes/xarm7_1305/collision/link3.stl; visual mesh filename=meshes/xarm7_1305/visual_glb/link3.glb
- link link4: geometry collision mesh filename=meshes/xarm7_1305/collision/link4.stl; visual mesh filename=meshes/xarm7_1305/visual_glb/link4.glb
- link link5: geometry collision mesh filename=meshes/xarm7_1305/collision/link5.stl; visual mesh filename=meshes/xarm7_1305/visual_glb/link5.glb
- link link6: geometry collision mesh filename=meshes/xarm7_1305/collision/link6.stl; visual mesh filename=meshes/xarm7_1305/visual_glb/link6.glb
- link link7: geometry collision mesh filename=meshes/xarm7_1305/collision/link7.stl; visual mesh filename=meshes/xarm7_1305/visual_glb/link7.glb
- link link_base: geometry collision mesh filename=meshes/xarm7_1305/collision/link_base.stl; visual mesh filename=meshes/xarm7_1305/visual_glb/link_base.glb

File: assets/urdf/xarm7/xarm7_1305_visual.glb.urdf (robot description, URDF)
Before this commit: robot gen, 9 links, 8 joints
Links:
- link link1: geometry collision mesh filename=meshes/xarm7_1305/collision/link1.stl; visual mesh filename=meshes/xarm7_1305/visual_glb/link1.glb
- link link2: geometry collision mesh filename=meshes/xarm7_1305/collision/link2.stl; visual mesh filename=meshes/xarm7_1305/visual_glb/link2.glb
- link link3: geometry collision mesh filename=meshes/xarm7_1305/collision/link3.stl; visual mesh filename=meshes/xarm7_1305/visual_glb/link3.glb
- link link4: geometry collision mesh filename=meshes/xarm7_1305/collision/link4.stl; visual mesh filename=meshes/xarm7_1305/visual_glb/link4.glb
- link link5: geometry collision mesh filename=meshes/xarm7_1305/collision/link5.stl; visual mesh filename=meshes/xarm7_1305/visual_glb/link5.glb
- link link6: geometry collision mesh filename=meshes/xarm7_1305/collision/link6.stl; visual mesh filename=meshes/xarm7_1305/visual_glb/link6.glb
- link link7: geometry collision mesh filename=meshes/xarm7_1305/collision/link7.stl; visual mesh filename=meshes/xarm7_1305/visual_glb/link7.glb
- link link_base: geometry collision mesh filename=meshes/xarm7_1305/collision/link_base.stl; visual mesh filename=meshes/xarm7_1305/visual_glb/link_base.glb
