Commit message: Fix Bio Gripper G2 arm mount and default xArm models to XI1305.
Compute per-robot bio_gripper_g2_attach from canonical EE pin-hole alignment
(fixes UF850 flange inversion and finger +X), regenerate combo URDFs/GLBs,
and add BioGripperG2 controller module. Resolve xarm5/6/7 short names to
*_1305 profiles with updated docs and registry tests.

Co-authored-by: Cursor <cursoragent@cursor.com>

File: assets/urdf/bio_gripper_g2/bio_gripper_g2.urdf (robot description, URDF)
Before this commit: robot bio_gripper_g2, 4 links, 4 joints
Joints:
- joint bio_gripper_g2_left_finger_joint: limit lower=-0.04 upper=0.0 effort=2.0 velocity=0.1 -> lower=-0.0395 upper=0.0 effort=2.0 velocity=0.1
- joint bio_gripper_g2_right_finger_joint: limit lower=0 upper=0.04 effort=2.0 velocity=0.1 -> lower=0 upper=0.0395 effort=2.0 velocity=0.1

File: assets/urdf/bio_gripper_g2/bio_gripper_g2_movable_visual.urdf (robot description, URDF)
Before this commit: robot bio_gripper_g2_movable_visual, 5 links, 4 joints
Joints:
- joint bio_gripper_g2_left_finger_joint: limit lower=-0.04 upper=0.0 effort=2.0 velocity=0.1 -> lower=-0.0395 upper=0.0 effort=2.0 velocity=0.1
- joint bio_gripper_g2_right_finger_joint: limit lower=0 upper=0.04 effort=2.0 velocity=0.1 -> lower=0 upper=0.0395 effort=2.0 velocity=0.1

File: assets/urdf/uf850/uf850_bio_gripper_g2_movable_visual.glb.urdf (robot description, URDF)
Before this commit: robot uf850_bio_gripper_g2_movable_visual.glb, 12 links, 11 joints
Joints:
- joint bio_gripper_g2_attach: origin xyz=0 0 0 rpy=3.14159265 0 0 -> xyz=0.034285 0.000413 -0.001674 rpy=0.00018025 0.01490249 -0.00018304
- joint bio_gripper_g2_left_finger_joint: limit lower=-0.04 upper=0.0 effort=2.0 velocity=0.1 -> lower=-0.0395 upper=0.0 effort=2.0 velocity=0.1
- joint bio_gripper_g2_right_finger_joint: limit lower=0 upper=0.04 effort=2.0 velocity=0.1 -> lower=0 upper=0.0395 effort=2.0 velocity=0.1

File: assets/urdf/uf850/uf850_bio_gripper_g2_visual.glb.urdf (robot description, URDF)
Before this commit: robot uf850_bio_gripper_g2_visual.glb, 13 links, 12 joints
Joints:
- joint bio_gripper_g2_left_finger_joint: limit lower=-0.04 upper=0.0 effort=2.0 velocity=0.1 -> lower=-0.0395 upper=0.0 effort=2.0 velocity=0.1
- joint bio_gripper_g2_right_finger_joint: limit lower=0 upper=0.04 effort=2.0 velocity=0.1 -> lower=0 upper=0.0395 effort=2.0 velocity=0.1

File: assets/urdf/xarm5/xarm5_1305_bio_gripper_g2_movable_visual.glb.urdf (robot description, URDF)
Before this commit: robot xarm5_1305_bio_gripper_g2_movable_visual.glb, 11 links, 10 joints
Joints:
- joint bio_gripper_g2_attach: origin xyz=0 0 0 rpy=3.14159265 0 0 -> xyz=0.026044 -0.000488 -0.000697 rpy=0.00000000 0.00000000 0.00702875
- joint bio_gripper_g2_left_finger_joint: limit lower=-0.04 upper=0.0 effort=2.0 velocity=0.1 -> lower=-0.0395 upper=0.0 effort=2.0 velocity=0.1
- joint bio_gripper_g2_right_finger_joint: limit lower=0 upper=0.04 effort=2.0 velocity=0.1 -> lower=0 upper=0.0395 effort=2.0 velocity=0.1

File: assets/urdf/xarm5/xarm5_1305_bio_gripper_g2_visual.glb.urdf (robot description, URDF)
Before this commit: robot xarm5_1305_bio_gripper_g2_visual.glb, 12 links, 11 joints
Joints:
- joint bio_gripper_g2_left_finger_joint: limit lower=-0.04 upper=0.0 effort=2.0 velocity=0.1 -> lower=-0.0395 upper=0.0 effort=2.0 velocity=0.1
- joint bio_gripper_g2_right_finger_joint: limit lower=0 upper=0.04 effort=2.0 velocity=0.1 -> lower=0 upper=0.0395 effort=2.0 velocity=0.1

File: assets/urdf/xarm6/xarm6_1305_bio_gripper_g2_movable_visual.glb.urdf (robot description, URDF)
Before this commit: robot xarm6_1305_bio_gripper_g2_movable_visual.glb, 13 links, 12 joints
Joints:
- joint bio_gripper_g2_attach: origin xyz=0 0 0 rpy=3.14159265 0 0 -> xyz=0.027018 -0.000335 -0.000692 rpy=0.00000000 0.00000000 0.00706128
- joint bio_gripper_g2_left_finger_joint: limit lower=-0.04 upper=0.0 effort=2.0 velocity=0.1 -> lower=-0.0395 upper=0.0 effort=2.0 velocity=0.1
- joint bio_gripper_g2_right_finger_joint: limit lower=0 upper=0.04 effort=2.0 velocity=0.1 -> lower=0 upper=0.0395 effort=2.0 velocity=0.1

File: assets/urdf/xarm6/xarm6_1305_bio_gripper_g2_visual.glb.urdf (robot description, URDF)
Before this commit: robot xarm6_1305_bio_gripper_g2_visual.glb, 14 links, 13 joints
Joints:
- joint bio_gripper_g2_left_finger_joint: limit lower=-0.04 upper=0.0 effort=2.0 velocity=0.1 -> lower=-0.0395 upper=0.0 effort=2.0 velocity=0.1
- joint bio_gripper_g2_right_finger_joint: limit lower=0 upper=0.04 effort=2.0 velocity=0.1 -> lower=0 upper=0.0395 effort=2.0 velocity=0.1

File: assets/urdf/xarm7/xarm7_1305_bio_gripper_g2_movable_visual.glb.urdf (robot description, URDF)
Before this commit: robot xarm7_1305_bio_gripper_g2_movable_visual.glb, 13 links, 12 joints
Joints:
- joint bio_gripper_g2_attach: origin xyz=0 0 0 rpy=3.14159265 0 0 -> xyz=0.026931 -0.000459 -0.000760 rpy=0.00000000 0.00000000 0.00784664
- joint bio_gripper_g2_left_finger_joint: limit lower=-0.04 upper=0.0 effort=2.0 velocity=0.1 -> lower=-0.0395 upper=0.0 effort=2.0 velocity=0.1
- joint bio_gripper_g2_right_finger_joint: limit lower=0 upper=0.04 effort=2.0 velocity=0.1 -> lower=0 upper=0.0395 effort=2.0 velocity=0.1

File: assets/urdf/xarm7/xarm7_1305_bio_gripper_g2_visual.glb.urdf (robot description, URDF)
Before this commit: robot xarm7_1305_bio_gripper_g2_visual.glb, 14 links, 13 joints
Joints:
- joint bio_gripper_g2_left_finger_joint: limit lower=-0.04 upper=0.0 effort=2.0 velocity=0.1 -> lower=-0.0395 upper=0.0 effort=2.0 velocity=0.1
- joint bio_gripper_g2_right_finger_joint: limit lower=0 upper=0.04 effort=2.0 velocity=0.1 -> lower=0 upper=0.0395 effort=2.0 velocity=0.1
