Commit message: Release v0.2.1: LSPB trajectory grasp-place and visual STL collision.
Add robot-aware LSPB planning, five-robot shared grasp-place examples,
Lite6 gripper gap modeling, and arm/accessory visual STL collision meshes.
Fix viewer startup pose and Lite6 finger-cube alignment in simulation.

Co-authored-by: Cursor <cursoragent@cursor.com>

File: assets/urdf/bio_gripper_g2/bio_gripper_g2.urdf (robot description, URDF)
Before this commit: robot bio_gripper_g2, 4 links, 4 joints
Links:
- link bio_gripper_g2_base_link: geometry collision mesh filename=meshes/visual/bio_gripper_g2_link_base.stl; visual mesh filename=meshes/visual/bio_gripper_g2_link_base.stl
- link bio_gripper_g2_left_finger: geometry collision mesh filename=meshes/visual/bio_gripper_g2_left_finger.stl; visual mesh filename=meshes/visual/bio_gripper_g2_left_finger.stl
- link bio_gripper_g2_right_finger: geometry collision mesh filename=meshes/visual/bio_gripper_g2_right_finger.stl; visual mesh filename=meshes/visual/bio_gripper_g2_right_finger.stl

File: assets/urdf/bio_gripper_g2/bio_gripper_g2_movable_visual.urdf (robot description, URDF)
Before this commit: robot bio_gripper_g2_movable_visual, 5 links, 4 joints
Links:
- link bio_gripper_g2_base_link: geometry collision mesh filename=../bio_gripper_g2/meshes/visual/bio_gripper_g2_link_base.stl; visual mesh filename=../bio_gripper_g2/meshes/visual/visual_glb/link6/bio_grippe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
- link bio_gripper_g2_left_finger: geometry collision mesh filename=../bio_gripper_g2/meshes/visual/bio_gripper_g2_left_finger.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; visual mesh filename=../bio_gripper_g2/meshes/visual/visual_glb/link6/bio_grippe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
- link bio_gripper_g2_right_finger: geometry collision mesh filename=../bio_gripper_g2/meshes/visual/bio_gripper_g2_right_finger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; visual mesh filename=../bio_gripper_g2/meshes/visual/visual_glb/link6/bio_grippe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

File: assets/urdf/lite6/lite6.urdf (robot description, URDF)
Before this commit: robot gen, 8 links, 7 joints
Links:
- link link1: geometry collision mesh filename=meshes/lite6/visual/link1.stl; visual mesh filename=meshes/lite6/visual/link1.stl
- link link2: geometry collision mesh filename=meshes/lite6/visual/link2.stl; visual mesh filename=meshes/lite6/visual/link2.stl
- link link3: geometry collision mesh filename=meshes/lite6/visual/link3.stl; visual mesh filename=meshes/lite6/visual/link3.stl
- link link4: geometry collision mesh filename=meshes/lite6/visual/link4.stl; visual mesh filename=meshes/lite6/visual/link4.stl
- link link5: geometry collision mesh filename=meshes/lite6/visual/link5.stl; visual mesh filename=meshes/lite6/visual/link5.stl
- link link6: geometry collision mesh filename=meshes/lite6/visual/link6.stl; visual mesh filename=meshes/lite6/visual/link6.stl
- link link_base: geometry collision mesh filename=meshes/lite6/visual/link_base.stl; visual mesh filename=meshes/lite6/visual/link_base.stl

File: assets/urdf/lite6/lite6_gripper_movable_visual.glb.urdf (robot description, URDF)
Before this commit: robot lite6_gripper_movable_visual.glb, 12 links, 11 joints
Links:
- link link1: geometry collision mesh filename=meshes/lite6/visual/link1.stl; visual mesh filename=meshes/lite6/visual_glb/link1.glb
- link link2: geometry collision mesh filename=meshes/lite6/visual/link2.stl; visual mesh filename=meshes/lite6/visual_glb/link2.glb
- link link3: geometry collision mesh filename=meshes/lite6/visual/link3.stl; visual mesh filename=meshes/lite6/visual_glb/link3.glb
- link link4: geometry collision mesh filename=meshes/lite6/visual/link4.stl; visual mesh filename=meshes/lite6/visual_glb/link4.glb
- link link5: geometry collision mesh filename=meshes/lite6/visual/link5.stl; visual mesh filename=meshes/lite6/visual_glb/link5.glb
- link link6: geometry collision mesh filename=meshes/lite6/visual/link6.stl; visual mesh filename=meshes/lite6/visual_glb/link6.glb
- link link_base: geometry collision mesh filename=meshes/lite6/visual/link_base.stl; visual mesh filename=meshes/lite6/visual_glb/link_base.glb
- link uflite_finger1: geometry collision mesh filename=../lite6_gripper/meshes/collision/finger1.stl; visual mesh filename=../lite6_gripper/meshes/collision/finger1.stl
- link uflite_finger2: geometry collision mesh filename=../lite6_gripper/meshes/collision/finger2.stl; visual mesh filename=../lite6_gripper/meshes/collision/finger2.stl

File: assets/urdf/lite6/lite6_gripper_visual.glb.urdf (robot description, URDF)
Before this commit: robot lite6_gripper_visual.glb, 13 links, 12 joints
Links:
- link link1: geometry collision mesh filename=meshes/lite6/visual/link1.stl; visual mesh filename=meshes/lite6/visual_glb/link1.glb
- link link2: geometry collision mesh filename=meshes/lite6/visual/link2.stl; visual mesh filename=meshes/lite6/visual_glb/link2.glb
- link link3: geometry collision mesh filename=meshes/lite6/visual/link3.stl; visual mesh filename=meshes/lite6/visual_glb/link3.glb
- link link4: geometry collision mesh filename=meshes/lite6/visual/link4.stl; visual mesh filename=meshes/lite6/visual_glb/link4.glb
- link link5: geometry collision mesh filename=meshes/lite6/visual/link5.stl; visual mesh filename=meshes/lite6/visual_glb/link5.glb
- link link6: geometry collision mesh filename=meshes/lite6/visual/link6.stl; visual mesh filename=meshes/lite6/visual_glb/link6.glb
- link link_base: geometry collision mesh filename=meshes/lite6/visual/link_base.stl; visual mesh filename=meshes/lite6/visual_glb/link_base.glb

File: assets/urdf/lite6/lite6_vacuum_gripper_visual.glb.urdf (robot description, URDF)
Before this commit: robot lite6_vacuum_gripper_visual.glb, 9 links, 8 joints
Links:
- link link1: geometry collision mesh filename=meshes/lite6/visual/link1.stl; visual mesh filename=meshes/lite6/visual_glb/link1.glb
- link link2: geometry collision mesh filename=meshes/lite6/visual/link2.stl; visual mesh filename=meshes/lite6/visual_glb/link2.glb
- link link3: geometry collision mesh filename=meshes/lite6/visual/link3.stl; visual mesh filename=meshes/lite6/visual_glb/link3.glb
- link link4: geometry collision mesh filename=meshes/lite6/visual/link4.stl; visual mesh filename=meshes/lite6/visual_glb/link4.glb
- link link5: geometry collision mesh filename=meshes/lite6/visual/link5.stl; visual mesh filename=meshes/lite6/visual_glb/link5.glb
- link link6: geometry collision mesh filename=meshes/lite6/visual/link6.stl; visual mesh filename=meshes/lite6/visual_glb/link6.glb
- link link_base: geometry collision mesh filename=meshes/lite6/visual/link_base.stl; visual mesh filename=meshes/lite6/visual_glb/link_base.glb
- link lite6_vacuum_gripper_visual: geometry collision mesh filename=../lite6_vacuum_gripper/meshes/visual/vacuum_gripper_lite.s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; visual mesh filename=../lite6_vacuum_gripper/meshes/visual/lite6_vacuum_gripper_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

File: assets/urdf/lite6/lite6_visual.glb.urdf (robot description, URDF)
Before this commit: robot gen, 8 links, 7 joints
Links:
- link link1: geometry collision mesh filename=meshes/lite6/visual/link1.stl; visual mesh filename=meshes/lite6/visual_glb/link1.glb
- link link2: geometry collision mesh filename=meshes/lite6/visual/link2.stl; visual mesh filename=meshes/lite6/visual_glb/link2.glb
- link link3: geometry collision mesh filename=meshes/lite6/visual/link3.stl; visual mesh filename=meshes/lite6/visual_glb/link3.glb
- link link4: geometry collision mesh filename=meshes/lite6/visual/link4.stl; visual mesh filename=meshes/lite6/visual_glb/link4.glb
- link link5: geometry collision mesh filename=meshes/lite6/visual/link5.stl; visual mesh filename=meshes/lite6/visual_glb/link5.glb
- link link6: geometry collision mesh filename=meshes/lite6/visual/link6.stl; visual mesh filename=meshes/lite6/visual_glb/link6.glb
- link link_base: geometry collision mesh filename=meshes/lite6/visual/link_base.stl; visual mesh filename=meshes/lite6/visual_glb/link_base.glb

File: assets/urdf/lite6/lite6_with_gripper.urdf (robot description, URDF)
Before this commit: robot lite6_with_gripper, 12 links, 11 joints
Links:
- link link1: geometry collision mesh filename=meshes/lite6/visual/link1.stl; visual mesh filename=meshes/lite6/visual/link1.stl
- link link2: geometry collision mesh filename=meshes/lite6/visual/link2.stl; visual mesh filename=meshes/lite6/visual/link2.stl
- link link3: geometry collision mesh filename=meshes/lite6/visual/link3.stl; visual mesh filename=meshes/lite6/visual/link3.stl
- link link4: geometry collision mesh filename=meshes/lite6/visual/link4.stl; visual mesh filename=meshes/lite6/visual/link4.stl
- link link5: geometry collision mesh filename=meshes/lite6/visual/link5.stl; visual mesh filename=meshes/lite6/visual/link5.stl
- link link6: geometry collision mesh filename=meshes/lite6/visual/link6.stl; visual mesh filename=meshes/lite6/visual/link6.stl
- link link_base: geometry collision mesh filename=meshes/lite6/visual/link_base.stl; visual mesh filename=meshes/lite6/visual/link_base.stl

File: assets/urdf/lite6/lite6_with_vacuum_gripper.urdf (robot description, URDF)
Before this commit: robot lite6_with_vacuum_gripper, 10 links, 9 joints
Links:
- link link1: geometry collision mesh filename=meshes/lite6/visual/link1.stl; visual mesh filename=meshes/lite6/visual/link1.stl
- link link2: geometry collision mesh filename=meshes/lite6/visual/link2.stl; visual mesh filename=meshes/lite6/visual/link2.stl
- link link3: geometry collision mesh filename=meshes/lite6/visual/link3.stl; visual mesh filename=meshes/lite6/visual/link3.stl
- link link4: geometry collision mesh filename=meshes/lite6/visual/link4.stl; visual mesh filename=meshes/lite6/visual/link4.stl
- link link5: geometry collision mesh filename=meshes/lite6/visual/link5.stl; visual mesh filename=meshes/lite6/visual/link5.stl
- link link6: geometry collision mesh filename=meshes/lite6/visual/link6.stl; visual mesh filename=meshes/lite6/visual/link6.stl
- link link_base: geometry collision mesh filename=meshes/lite6/visual/link_base.stl; visual mesh filename=meshes/lite6/visual/link_base.stl
- link uflite_vacuum_gripper_link: geometry collision mesh filename=../lite6_vacuum_gripper/meshes/visual/vacuum_gripper_lite.s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; visual mesh filename=../lite6_vacuum_gripper/meshes/visual/vacuum_gripper_lite.s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

File: assets/urdf/lite6_gripper/lite6_gripper_movable_visual.urdf (robot description, URDF)
Before this commit: robot lite6_gripper_movable_visual, 5 links, 4 joints
Links:
- link uflite_finger1: geometry collision mesh filename=../lite6_gripper/meshes/collision/finger1.stl; visual mesh filename=../lite6_gripper/meshes/collision/finger1.stl
- link uflite_finger2: geometry collision mesh filename=../lite6_gripper/meshes/collision/finger2.stl; visual mesh filename=../lite6_gripper/meshes/collision/finger2.stl

File: assets/urdf/lite6_vacuum_gripper/lite6_vacuum_gripper.urdf (robot description, URDF)
Before this commit: robot lite6_vacuum_gripper, 2 links, 2 joints
Links:
- link uflite_vacuum_gripper_link: geometry collision mesh filename=meshes/visual/vacuum_gripper_lite.stl; visual mesh filename=meshes/visual/vacuum_gripper_lite.stl

File: assets/urdf/uf850/uf850.urdf (robot description, URDF)
Before this commit: robot gen, 8 links, 7 joints
Links:
- link link1: geometry collision mesh filename=meshes/uf850/visual/link1.stl; visual mesh filename=meshes/uf850/visual/link1.stl
- link link2: geometry collision mesh filename=meshes/uf850/visual/link2.stl; visual mesh filename=meshes/uf850/visual/link2.stl
- link link3: geometry collision mesh filename=meshes/uf850/visual/link3.stl; visual mesh filename=meshes/uf850/visual/link3.stl
- link link4: geometry collision mesh filename=meshes/uf850/visual/link4.stl; visual mesh filename=meshes/uf850/visual/link4.stl
- link link5: geometry collision mesh filename=meshes/uf850/visual/link5.stl; visual mesh filename=meshes/uf850/visual/link5.stl
- link link6: geometry collision mesh filename=meshes/uf850/visual/link6.stl; visual mesh filename=meshes/uf850/visual/link6.stl
- link link_base: geometry collision mesh filename=meshes/uf850/visual/link_base.stl; visual mesh filename=meshes/uf850/visual/link_base.stl

File: assets/urdf/uf850/uf850_bio_gripper_g2_movable_visual.glb.urdf (robot description, URDF)
Before this commit: robot uf850_bio_gripper_g2_movable_visual.glb, 12 links, 11 joints
Links:
- link bio_gripper_g2_base_link: geometry collision mesh filename=../bio_gripper_g2/meshes/visual/bio_gripper_g2_link_base.stl; visual mesh filename=../bio_gripper_g2/meshes/visual/visual_glb/link6/bio_grippe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
- link bio_gripper_g2_left_finger: geometry collision mesh filename=../bio_gripper_g2/meshes/visual/bio_gripper_g2_left_finger.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; visual mesh filename=../bio_gripper_g2/meshes/visual/visual_glb/link6/bio_grippe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
- link bio_gripper_g2_right_finger: geometry collision mesh filename=../bio_gripper_g2/meshes/visual/bio_gripper_g2_right_finger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; visual mesh filename=../bio_gripper_g2/meshes/visual/visual_glb/link6/bio_grippe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
- link link1: geometry collision mesh filename=meshes/uf850/visual/link1.stl; visual mesh filename=meshes/uf850/visual_glb/link1.glb
- link link2: geometry collision mesh filename=meshes/uf850/visual/link2.stl; visual mesh filename=meshes/uf850/visual_glb/link2.glb
- link link3: geometry collision mesh filename=meshes/uf850/visual/link3.stl; visual mesh filename=meshes/uf850/visual_glb/link3.glb
- link link4: geometry collision mesh filename=meshes/uf850/visual/link4.stl; visual mesh filename=meshes/uf850/visual_glb/link4.glb
- link link5: geometry collision mesh filename=meshes/uf850/visual/link5.stl; visual mesh filename=meshes/uf850/visual_glb/link5.glb
- link link6: geometry collision mesh filename=meshes/uf850/visual/link6.stl; visual mesh filename=meshes/uf850/visual_glb/link6.glb
- link link_base: geometry collision mesh filename=meshes/uf850/visual/link_base.stl; visual mesh filename=meshes/uf850/visual_glb/link_base.glb

File: assets/urdf/uf850/uf850_bio_gripper_g2_visual.glb.urdf (robot description, URDF)
Before this commit: robot uf850_bio_gripper_g2_visual.glb, 13 links, 12 joints
Links:
- link bio_gripper_g2_base_link: geometry collision mesh filename=../bio_gripper_g2/meshes/visual/bio_gripper_g2_link_base.stl
- link bio_gripper_g2_left_finger: geometry collision mesh filename=../bio_gripper_g2/meshes/visual/bio_gripper_g2_left_finger.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
- link bio_gripper_g2_right_finger: geometry collision mesh filename=../bio_gripper_g2/meshes/visual/bio_gripper_g2_right_finger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
- link link1: geometry collision mesh filename=meshes/uf850/visual/link1.stl; visual mesh filename=meshes/uf850/visual_glb/link1.glb
- link link2: geometry collision mesh filename=meshes/uf850/visual/link2.stl; visual mesh filename=meshes/uf850/visual_glb/link2.glb
- link link3: geometry collision mesh filename=meshes/uf850/visual/link3.stl; visual mesh filename=meshes/uf850/visual_glb/link3.glb
- link link4: geometry collision mesh filename=meshes/uf850/visual/link4.stl; visual mesh filename=meshes/uf850/visual_glb/link4.glb
- link link5: geometry collision mesh filename=meshes/uf850/visual/link5.stl; visual mesh filename=meshes/uf850/visual_glb/link5.glb
- link link6: geometry collision mesh filename=meshes/uf850/visual/link6.stl; visual mesh filename=meshes/uf850/visual_glb/link6.glb
- link link_base: geometry collision mesh filename=meshes/uf850/visual/link_base.stl; visual mesh filename=meshes/uf850/visual_glb/link_base.glb

File: assets/urdf/uf850/uf850_g2_movable_visual.urdf (robot description, URDF)
Before this commit: robot uf850_g2_movable_visual, 16 links, 15 joints
Links:
- link link1: geometry collision mesh filename=meshes/uf850/visual/link1.stl; visual mesh filename=meshes/uf850/visual_glb/link1.glb
- link link2: geometry collision mesh filename=meshes/uf850/visual/link2.stl; visual mesh filename=meshes/uf850/visual_glb/link2.glb
- link link3: geometry collision mesh filename=meshes/uf850/visual/link3.stl; visual mesh filename=meshes/uf850/visual_glb/link3.glb
- link link4: geometry collision mesh filename=meshes/uf850/visual/link4.stl; visual mesh filename=meshes/uf850/visual_glb/link4.glb
- link link5: geometry collision mesh filename=meshes/uf850/visual/link5.stl; visual mesh filename=meshes/uf850/visual_glb/link5.glb
- link link6: geometry collision mesh filename=meshes/uf850/visual/link6.stl; visual mesh filename=meshes/uf850/visual_glb/link6.glb
- link link_base: geometry collision mesh filename=meshes/uf850/visual/link_base.stl; visual mesh filename=meshes/uf850/visual_glb/link_base.glb

File: assets/urdf/uf850/uf850_g2_visual.urdf (robot description, URDF)
Before this commit: robot uf850_g2_visual, 17 links, 16 joints
Links:
- link link1: geometry collision mesh filename=meshes/uf850/visual/link1.stl; visual mesh filename=meshes/uf850/visual_glb/link1.glb
- link link2: geometry collision mesh filename=meshes/uf850/visual/link2.stl; visual mesh filename=meshes/uf850/visual_glb/link2.glb
- link link3: geometry collision mesh filename=meshes/uf850/visual/link3.stl; visual mesh filename=meshes/uf850/visual_glb/link3.glb
- link link4: geometry collision mesh filename=meshes/uf850/visual/link4.stl; visual mesh filename=meshes/uf850/visual_glb/link4.glb
- link link5: geometry collision mesh filename=meshes/uf850/visual/link5.stl; visual mesh filename=meshes/uf850/visual_glb/link5.glb
- link link6: geometry collision mesh filename=meshes/uf850/visual/link6.stl; visual mesh filename=meshes/uf850/visual_glb/link6.glb
- link link_base: geometry collision mesh filename=meshes/uf850/visual/link_base.stl; visual mesh filename=meshes/uf850/visual_glb/link_base.glb

File: assets/urdf/uf850/uf850_visual.glb.urdf (robot description, URDF)
Before this commit: robot gen, 8 links, 7 joints
Links:
- link link1: geometry collision mesh filename=meshes/uf850/visual/link1.stl; visual mesh filename=meshes/uf850/visual_glb/link1.glb
- link link2: geometry collision mesh filename=meshes/uf850/visual/link2.stl; visual mesh filename=meshes/uf850/visual_glb/link2.glb
- link link3: geometry collision mesh filename=meshes/uf850/visual/link3.stl; visual mesh filename=meshes/uf850/visual_glb/link3.glb
- link link4: geometry collision mesh filename=meshes/uf850/visual/link4.stl; visual mesh filename=meshes/uf850/visual_glb/link4.glb
- link link5: geometry collision mesh filename=meshes/uf850/visual/link5.stl; visual mesh filename=meshes/uf850/visual_glb/link5.glb
- link link6: geometry collision mesh filename=meshes/uf850/visual/link6.stl; visual mesh filename=meshes/uf850/visual_glb/link6.glb
- link link_base: geometry collision mesh filename=meshes/uf850/visual/link_base.stl; visual mesh filename=meshes/uf850/visual_glb/link_base.glb

File: assets/urdf/xarm5/xarm5_1305.urdf (robot description, URDF)
Before this commit: robot gen, 7 links, 6 joints
Links:
- link link1: geometry collision mesh filename=meshes/xarm5_1305/visual/link1.stl; visual mesh filename=meshes/xarm5_1305/visual/link1.stl
- link link2: geometry collision mesh filename=meshes/xarm5_1305/visual/link2.stl; visual mesh filename=meshes/xarm5_1305/visual/link2.stl
- link link3: geometry collision mesh filename=meshes/xarm5_1305/visual/link3.stl; visual mesh filename=meshes/xarm5_1305/visual/link3.stl
- link link4: geometry collision mesh filename=meshes/xarm5_1305/visual/link4.stl; visual mesh filename=meshes/xarm5_1305/visual/link4.stl
- link link5: geometry collision mesh filename=meshes/xarm5_1305/visual/link5.stl; visual mesh filename=meshes/xarm5_1305/visual/link5.stl
- link link_base: geometry collision mesh filename=meshes/xarm5_1305/visual/link_base.stl; visual mesh filename=meshes/xarm5_1305/visual/link_base.stl

File: assets/urdf/xarm5/xarm5_1305_bio_gripper_g2_movable_visual.glb.urdf (robot description, URDF)
Before this commit: robot xarm5_1305_bio_gripper_g2_movable_visual.glb, 11 links, 10 joints
Links:
- link bio_gripper_g2_base_link: geometry collision mesh filename=../bio_gripper_g2/meshes/visual/bio_gripper_g2_link_base.stl; visual mesh filename=../bio_gripper_g2/meshes/visual/visual_glb/link5/bio_grippe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
- link bio_gripper_g2_left_finger: geometry collision mesh filename=../bio_gripper_g2/meshes/visual/bio_gripper_g2_left_finger.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; visual mesh filename=../bio_gripper_g2/meshes/visual/visual_glb/link5/bio_grippe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
- link bio_gripper_g2_right_finger: geometry collision mesh filename=../bio_gripper_g2/meshes/visual/bio_gripper_g2_right_finger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; visual mesh filename=../bio_gripper_g2/meshes/visual/visual_glb/link5/bio_grippe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
- link link1: geometry collision mesh filename=meshes/xarm5_1305/visual/link1.stl; visual mesh filename=meshes/xarm5_1305/visual_glb/link1.glb
- link link2: geometry collision mesh filename=meshes/xarm5_1305/visual/link2.stl; visual mesh filename=meshes/xarm5_1305/visual_glb/link2.glb
- link link3: geometry collision mesh filename=meshes/xarm5_1305/visual/link3.stl; visual mesh filename=meshes/xarm5_1305/visual_glb/link3.glb
- link link4: geometry collision mesh filename=meshes/xarm5_1305/visual/link4.stl; visual mesh filename=meshes/xarm5_1305/visual_glb/link4.glb
- link link5: geometry collision mesh filename=meshes/xarm5_1305/visual/link5.stl; visual mesh filename=meshes/xarm5_1305/visual_glb/link5.glb
- link link_base: geometry collision mesh filename=meshes/xarm5_1305/visual/link_base.stl; visual mesh filename=meshes/xarm5_1305/visual_glb/link_base.glb

File: assets/urdf/xarm5/xarm5_1305_bio_gripper_g2_visual.glb.urdf (robot description, URDF)
Before this commit: robot xarm5_1305_bio_gripper_g2_visual.glb, 12 links, 11 joints
Links:
- link bio_gripper_g2_base_link: geometry collision mesh filename=../bio_gripper_g2/meshes/visual/bio_gripper_g2_link_base.stl
- link bio_gripper_g2_left_finger: geometry collision mesh filename=../bio_gripper_g2/meshes/visual/bio_gripper_g2_left_finger.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
- link bio_gripper_g2_right_finger: geometry collision mesh filename=../bio_gripper_g2/meshes/visual/bio_gripper_g2_right_finger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
- link link1: geometry collision mesh filename=meshes/xarm5_1305/visual/link1.stl; visual mesh filename=meshes/xarm5_1305/visual_glb/link1.glb
- link link2: geometry collision mesh filename=meshes/xarm5_1305/visual/link2.stl; visual mesh filename=meshes/xarm5_1305/visual_glb/link2.glb
- link link3: geometry collision mesh filename=meshes/xarm5_1305/visual/link3.stl; visual mesh filename=meshes/xarm5_1305/visual_glb/link3.glb
- link link4: geometry collision mesh filename=meshes/xarm5_1305/visual/link4.stl; visual mesh filename=meshes/xarm5_1305/visual_glb/link4.glb
- link link5: geometry collision mesh filename=meshes/xarm5_1305/visual/link5.stl; visual mesh filename=meshes/xarm5_1305/visual_glb/link5.glb
- link link_base: geometry collision mesh filename=meshes/xarm5_1305/visual/link_base.stl; visual mesh filename=meshes/xarm5_1305/visual_glb/link_base.glb
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