Commit message: Prepare v0.1.6 public release surface

File: assets/urdf/bio_gripper_g2/bio_gripper_g2.urdf (robot description, URDF)
Before this commit: robot bio_gripper_g2, 4 links, 4 joints
Links:
- link bio_gripper_g2_base_link: geometry collision mesh filename=meshes/visual/link_base.stl; visual mesh filename=meshes/visual/link_base.stl
- link bio_gripper_g2_left_finger: geometry collision mesh filename=meshes/visual/left_finger.stl; visual mesh filename=meshes/visual/left_finger.stl
- link bio_gripper_g2_right_finger: geometry collision mesh filename=meshes/visual/right_finger.stl; visual mesh filename=meshes/visual/right_finger.stl

File: assets/urdf/gripper_g2/gripper_g2.urdf (robot description, URDF)
Before this commit: robot gripper_g2, 8 links, 8 joints
Links:
- link left_finger: geometry collision mesh filename=meshes/collision/left_finger.stl; visual mesh filename=meshes/collision/left_finger.stl
- link left_inner_knuckle: geometry collision mesh filename=meshes/collision/left_inner_knuckle.stl; visual mesh filename=meshes/collision/left_inner_knuckle.stl
- link left_outer_knuckle: geometry collision mesh filename=meshes/collision/left_outer_knuckle.stl; visual mesh filename=meshes/collision/left_outer_knuckle.stl
- link right_finger: geometry collision mesh filename=meshes/collision/right_finger.stl; visual mesh filename=meshes/collision/right_finger.stl
- link right_inner_knuckle: geometry collision mesh filename=meshes/collision/right_inner_knuckle.stl; visual mesh filename=meshes/collision/right_inner_knuckle.stl
- link right_outer_knuckle: geometry collision mesh filename=meshes/collision/right_outer_knuckle.stl; visual mesh filename=meshes/collision/right_outer_knuckle.stl
- link xarm_gripper_base_link: geometry collision mesh filename=meshes/collision/base_link.stl; visual mesh filename=meshes/collision/base_link.stl

File: assets/urdf/xarm6/xarm6_1305.urdf (robot description, URDF)
Before this commit: robot xarm6_1305, 9 links, 8 joints
Links:
- link link1: geometry collision mesh filename=meshes/xarm6_1305/collision/link1.obj; visual mesh filename=meshes/xarm6_1305/visual/link1.stl
- link link2: geometry collision mesh filename=meshes/xarm6_1305/collision/link2.obj; visual mesh filename=meshes/xarm6_1305/visual/link2.stl
- link link3: geometry collision mesh filename=meshes/xarm6_1305/collision/link3.obj; visual mesh filename=meshes/xarm6_1305/visual/link3.stl
- link link4: geometry collision mesh filename=meshes/xarm6_1305/collision/link4.obj; visual mesh filename=meshes/xarm6_1305/visual/link4.stl
- link link5: geometry collision mesh filename=meshes/xarm6_1305/collision/link5.obj; visual mesh filename=meshes/xarm6_1305/visual/link5.stl
- link link6: geometry collision mesh filename=meshes/xarm6_1305/collision/link6.obj; visual mesh filename=meshes/xarm6_1305/visual/link6.stl
- link link_base: geometry collision mesh filename=meshes/xarm6_1305/collision/link_base.obj; visual mesh filename=meshes/xarm6_1305/visual/link_base.stl

File: assets/urdf/xarm6/xarm6_1305_bio_gripper_g2_movable_visual.glb.urdf (robot description, URDF)
Before this commit: robot xarm6_1305_bio_gripper_g2_movable_visual.glb, 13 links, 12 joints
Links:
- link link1: geometry collision mesh filename=meshes/xarm6_1305/collision/link1.obj; visual mesh filename=meshes/xarm6_1305/visual_glb/link1.glb
- link link2: geometry collision mesh filename=meshes/xarm6_1305/collision/link2.obj; visual mesh filename=meshes/xarm6_1305/visual_glb/link2.glb
- link link3: geometry collision mesh filename=meshes/xarm6_1305/collision/link3.obj; visual mesh filename=meshes/xarm6_1305/visual_glb/link3.glb
- link link4: geometry collision mesh filename=meshes/xarm6_1305/collision/link4.obj; visual mesh filename=meshes/xarm6_1305/visual_glb/link4.glb
- link link5: geometry collision mesh filename=meshes/xarm6_1305/collision/link5.obj; visual mesh filename=meshes/xarm6_1305/visual_glb/link5.glb
- link link6: geometry collision mesh filename=meshes/xarm6_1305/collision/link6.obj; visual mesh filename=meshes/xarm6_1305/visual_glb/link6.glb
- link link_base: geometry collision mesh filename=meshes/xarm6_1305/collision/link_base.obj; visual mesh filename=meshes/xarm6_1305/visual_glb/link_base.glb

File: assets/urdf/xarm6/xarm6_1305_bio_gripper_g2_visual.glb.urdf (robot description, URDF)
Before this commit: robot xarm6_1305_bio_gripper_g2_visual.glb, 14 links, 13 joints
Links:
- link link1: geometry collision mesh filename=meshes/xarm6_1305/collision/link1.obj; visual mesh filename=meshes/xarm6_1305/visual_glb/link1.glb
- link link2: geometry collision mesh filename=meshes/xarm6_1305/collision/link2.obj; visual mesh filename=meshes/xarm6_1305/visual_glb/link2.glb
- link link3: geometry collision mesh filename=meshes/xarm6_1305/collision/link3.obj; visual mesh filename=meshes/xarm6_1305/visual_glb/link3.glb
- link link4: geometry collision mesh filename=meshes/xarm6_1305/collision/link4.obj; visual mesh filename=meshes/xarm6_1305/visual_glb/link4.glb
- link link5: geometry collision mesh filename=meshes/xarm6_1305/collision/link5.obj; visual mesh filename=meshes/xarm6_1305/visual_glb/link5.glb
- link link6: geometry collision mesh filename=meshes/xarm6_1305/collision/link6.obj; visual mesh filename=meshes/xarm6_1305/visual_glb/link6.glb
- link link_base: geometry collision mesh filename=meshes/xarm6_1305/collision/link_base.obj; visual mesh filename=meshes/xarm6_1305/visual_glb/link_base.glb

File: assets/urdf/xarm6/xarm6_1305_g2_movable_visual.urdf (robot description, URDF)
Before this commit: robot xarm6_1305_g2_movable_visual, 17 links, 16 joints
Links:
- link link1: geometry collision mesh filename=meshes/xarm6_1305/collision/link1.obj; visual mesh filename=meshes/xarm6_1305/visual_glb/link1.glb
- link link2: geometry collision mesh filename=meshes/xarm6_1305/collision/link2.obj; visual mesh filename=meshes/xarm6_1305/visual_glb/link2.glb
- link link3: geometry collision mesh filename=meshes/xarm6_1305/collision/link3.obj; visual mesh filename=meshes/xarm6_1305/visual_glb/link3.glb
- link link4: geometry collision mesh filename=meshes/xarm6_1305/collision/link4.obj; visual mesh filename=meshes/xarm6_1305/visual_glb/link4.glb
- link link5: geometry collision mesh filename=meshes/xarm6_1305/collision/link5.obj; visual mesh filename=meshes/xarm6_1305/visual_glb/link5.glb
- link link6: geometry collision mesh filename=meshes/xarm6_1305/collision/link6.obj; visual mesh filename=meshes/xarm6_1305/visual_glb/link6.glb
- link link_base: geometry collision mesh filename=meshes/xarm6_1305/collision/link_base.obj; visual mesh filename=meshes/xarm6_1305/visual_glb/link_base.glb

File: assets/urdf/xarm6/xarm6_1305_g2_visual.urdf (robot description, URDF)
Before this commit: robot xarm6_1305_g2_visual, 18 links, 17 joints
Links:
- link link1: geometry collision mesh filename=meshes/xarm6_1305/collision/link1.obj; visual mesh filename=meshes/xarm6_1305/visual_glb/link1.glb
- link link2: geometry collision mesh filename=meshes/xarm6_1305/collision/link2.obj; visual mesh filename=meshes/xarm6_1305/visual_glb/link2.glb
- link link3: geometry collision mesh filename=meshes/xarm6_1305/collision/link3.obj; visual mesh filename=meshes/xarm6_1305/visual_glb/link3.glb
- link link4: geometry collision mesh filename=meshes/xarm6_1305/collision/link4.obj; visual mesh filename=meshes/xarm6_1305/visual_glb/link4.glb
- link link5: geometry collision mesh filename=meshes/xarm6_1305/collision/link5.obj; visual mesh filename=meshes/xarm6_1305/visual_glb/link5.glb
- link link6: geometry collision mesh filename=meshes/xarm6_1305/collision/link6.obj; visual mesh filename=meshes/xarm6_1305/visual_glb/link6.glb
- link link_base: geometry collision mesh filename=meshes/xarm6_1305/collision/link_base.obj; visual mesh filename=meshes/xarm6_1305/visual_glb/link_base.glb

File: assets/urdf/xarm6/xarm6_1305_visual.glb.urdf (robot description, URDF)
Before this commit: robot xarm6_1305_visual_glb, 9 links, 8 joints
Links:
- link link1: geometry collision mesh filename=meshes/xarm6_1305/collision/link1.obj; visual mesh filename=meshes/xarm6_1305/visual_glb/link1.glb
- link link2: geometry collision mesh filename=meshes/xarm6_1305/collision/link2.obj; visual mesh filename=meshes/xarm6_1305/visual_glb/link2.glb
- link link3: geometry collision mesh filename=meshes/xarm6_1305/collision/link3.obj; visual mesh filename=meshes/xarm6_1305/visual_glb/link3.glb
- link link4: geometry collision mesh filename=meshes/xarm6_1305/collision/link4.obj; visual mesh filename=meshes/xarm6_1305/visual_glb/link4.glb
- link link5: geometry collision mesh filename=meshes/xarm6_1305/collision/link5.obj; visual mesh filename=meshes/xarm6_1305/visual_glb/link5.glb
- link link6: geometry collision mesh filename=meshes/xarm6_1305/collision/link6.obj; visual mesh filename=meshes/xarm6_1305/visual_glb/link6.glb
- link link_base: geometry collision mesh filename=meshes/xarm6_1305/collision/link_base.obj; visual mesh filename=meshes/xarm6_1305/visual_glb/link_base.glb

File: assets/urdf/xarm6/xarm6_with_gripper.urdf (robot description, URDF)
Before this commit: robot xarm6_with_gripper, 17 links, 16 joints
Links:
- link link1: geometry collision mesh filename=meshes/xarm6_1305/collision/link1.obj; visual mesh filename=meshes/xarm6_1305/visual/link1.stl
- link link2: geometry collision mesh filename=meshes/xarm6_1305/collision/link2.obj; visual mesh filename=meshes/xarm6_1305/visual/link2.stl
- link link3: geometry collision mesh filename=meshes/xarm6_1305/collision/link3.obj; visual mesh filename=meshes/xarm6_1305/visual/link3.stl
- link link4: geometry collision mesh filename=meshes/xarm6_1305/collision/link4.obj; visual mesh filename=meshes/xarm6_1305/visual/link4.stl
- link link5: geometry collision mesh filename=meshes/xarm6_1305/collision/link5.obj; visual mesh filename=meshes/xarm6_1305/visual/link5.stl
- link link6: geometry collision mesh filename=meshes/xarm6_1305/collision/link6.obj; visual mesh filename=meshes/xarm6_1305/visual/link6.stl
- link link_base: geometry collision mesh filename=meshes/xarm6_1305/collision/link_base.obj; visual mesh filename=meshes/xarm6_1305/visual/link_base.stl

Commit message: Add Bio Gripper G2 calibrated dynamics, convex collision meshes, and microplate pick-place simulation

File: assets/urdf/bio_gripper_g2/bio_gripper_g2.urdf (robot description, URDF)
Before this commit: robot bio_gripper_g2, 4 links, 4 joints
Links:
- link bio_gripper_g2_base_link: mass 0.38837 -> 0.765827; geometry collision mesh filename=meshes/collision/bio_gripper_g2_base_link_convex_0.stl; visual mesh filename=meshes/visual/bio_gripper_g2_link_base.stl
- link bio_gripper_g2_left_finger: geometry collision mesh filename=meshes/collision/bio_gripper_g2_left_finger_convex_0.stl; collision mesh filename=meshes/collision/bio_gripper_g2_left_finger_convex_1.stl
- link bio_gripper_g2_right_finger: geometry collision mesh filename=meshes/collision/bio_gripper_g2_right_finger_convex_0.stl; collision mesh filename=meshes/collision/bio_gripper_g2_right_finger_convex_1.stl
Joints:
- joint bio_gripper_g2_left_finger_joint: limit lower=-0.0395 upper=0.0 effort=2.0 velocity=0.1 -> lower=-0.0395 upper=0.0 effort=40 velocity=0.333333333333333
- joint bio_gripper_g2_right_finger_joint: limit lower=0 upper=0.0395 effort=2.0 velocity=0.1 -> lower=0 upper=0.0395 effort=40 velocity=0.333333333333333

File: assets/urdf/bio_gripper_g2/bio_gripper_g2_movable_visual.urdf (robot description, URDF)
Before this commit: robot bio_gripper_g2_movable_visual, 5 links, 4 joints
Links:
- link bio_gripper_g2_base_link: mass 0.38837 -> 0.765827; geometry collision mesh filename=../bio_gripper_g2/meshes/collision/bio_gripper_g2_base_link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; visual mesh filename=../bio_gripper_g2/meshes/visual/visual_glb/bio_gripper_g2_b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
- link bio_gripper_g2_left_finger: geometry collision mesh filename=../bio_gripper_g2/meshes/collision/bio_gripper_g2_left_fing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; collision mesh filename=../bio_gripper_g2/meshes/collision/bio_gripper_g2_left_fing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
- link bio_gripper_g2_right_finger: geometry collision mesh filename=../bio_gripper_g2/meshes/collision/bio_gripper_g2_right_fin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; collision mesh filename=../bio_gripper_g2/meshes/collision/bio_gripper_g2_right_fin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
Joints:
- joint bio_gripper_g2_left_finger_joint: limit lower=-0.0395 upper=0.0 effort=2.0 velocity=0.1 -> lower=-0.0395 upper=0.0 effort=40 velocity=0.333333333333333
- joint bio_gripper_g2_right_finger_joint: limit lower=0 upper=0.0395 effort=2.0 velocity=0.1 -> lower=0 upper=0.0395 effort=40 velocity=0.333333333333333

File: assets/urdf/uf850/uf850_bio_gripper_g2_movable_visual.glb.urdf (robot description, URDF)
Before this commit: robot uf850_bio_gripper_g2_movable_visual.glb, 12 links, 11 joints
Links:
- link bio_gripper_g2_base_link: mass 0.38837 -> 0.765827; geometry collision mesh filename=../bio_gripper_g2/meshes/collision/bio_gripper_g2_base_link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; visual mesh filename=../bio_gripper_g2/meshes/visual/visual_glb/bio_gripper_g2_b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
- link bio_gripper_g2_left_finger: geometry collision mesh filename=../bio_gripper_g2/meshes/collision/bio_gripper_g2_left_fing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; collision mesh filename=../bio_gripper_g2/meshes/collision/bio_gripper_g2_left_fing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
- link bio_gripper_g2_right_finger: geometry collision mesh filename=../bio_gripper_g2/meshes/collision/bio_gripper_g2_right_fin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; collision mesh filename=../bio_gripper_g2/meshes/collision/bio_gripper_g2_right_fin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
Joints:
- joint bio_gripper_g2_left_finger_joint: limit lower=-0.0395 upper=0.0 effort=2.0 velocity=0.1 -> lower=-0.0395 upper=0.0 effort=40 velocity=0.333333333333333
- joint bio_gripper_g2_right_finger_joint: limit lower=0 upper=0.0395 effort=2.0 velocity=0.1 -> lower=0 upper=0.0395 effort=40 velocity=0.333333333333333

File: assets/urdf/uf850/uf850_bio_gripper_g2_visual.glb.urdf (robot description, URDF)
Before this commit: robot uf850_bio_gripper_g2_visual.glb, 13 links, 12 joints
Links:
- link bio_gripper_g2_base_link: mass 0.38837 -> 0.765827; geometry collision mesh filename=../bio_gripper_g2/meshes/collision/bio_gripper_g2_base_link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
- link bio_gripper_g2_left_finger: geometry collision mesh filename=../bio_gripper_g2/meshes/collision/bio_gripper_g2_left_fing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; collision mesh filename=../bio_gripper_g2/meshes/collision/bio_gripper_g2_left_fing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
- link bio_gripper_g2_right_finger: geometry collision mesh filename=../bio_gripper_g2/meshes/collision/bio_gripper_g2_right_fin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; collision mesh filename=../bio_gripper_g2/meshes/collision/bio_gripper_g2_right_fin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
Joints:
- joint bio_gripper_g2_left_finger_joint: limit lower=-0.0395 upper=0.0 effort=2.0 velocity=0.1 -> lower=-0.0395 upper=0.0 effort=40 velocity=0.333333333333333
- joint bio_gripper_g2_right_finger_joint: limit lower=0 upper=0.0395 effort=2.0 velocity=0.1 -> lower=0 upper=0.0395 effort=40 velocity=0.333333333333333

File: assets/urdf/xarm5/xarm5_1305_bio_gripper_g2_movable_visual.glb.urdf (robot description, URDF)
Before this commit: robot xarm5_1305_bio_gripper_g2_movable_visual.glb, 11 links, 10 joints
Links:
- link bio_gripper_g2_base_link: mass 0.38837 -> 0.765827; geometry collision mesh filename=../bio_gripper_g2/meshes/collision/bio_gripper_g2_base_link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; visual mesh filename=../bio_gripper_g2/meshes/visual/visual_glb/bio_gripper_g2_b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
- link bio_gripper_g2_left_finger: geometry collision mesh filename=../bio_gripper_g2/meshes/collision/bio_gripper_g2_left_fing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; collision mesh filename=../bio_gripper_g2/meshes/collision/bio_gripper_g2_left_fing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
- link bio_gripper_g2_right_finger: geometry collision mesh filename=../bio_gripper_g2/meshes/collision/bio_gripper_g2_right_fin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; collision mesh filename=../bio_gripper_g2/meshes/collision/bio_gripper_g2_right_fin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
Joints:
- joint bio_gripper_g2_left_finger_joint: limit lower=-0.0395 upper=0.0 effort=2.0 velocity=0.1 -> lower=-0.0395 upper=0.0 effort=40 velocity=0.333333333333333
- joint bio_gripper_g2_right_finger_joint: limit lower=0 upper=0.0395 effort=2.0 velocity=0.1 -> lower=0 upper=0.0395 effort=40 velocity=0.333333333333333

File: assets/urdf/xarm5/xarm5_1305_bio_gripper_g2_visual.glb.urdf (robot description, URDF)
Before this commit: robot xarm5_1305_bio_gripper_g2_visual.glb, 12 links, 11 joints
Links:
- link bio_gripper_g2_base_link: mass 0.38837 -> 0.765827; geometry collision mesh filename=../bio_gripper_g2/meshes/collision/bio_gripper_g2_base_link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
- link bio_gripper_g2_left_finger: geometry collision mesh filename=../bio_gripper_g2/meshes/collision/bio_gripper_g2_left_fing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; collision mesh filename=../bio_gripper_g2/meshes/collision/bio_gripper_g2_left_fing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
- link bio_gripper_g2_right_finger: geometry collision mesh filename=../bio_gripper_g2/meshes/collision/bio_gripper_g2_right_fin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; collision mesh filename=../bio_gripper_g2/meshes/collision/bio_gripper_g2_right_fin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
Joints:
- joint bio_gripper_g2_left_finger_joint: limit lower=-0.0395 upper=0.0 effort=2.0 velocity=0.1 -> lower=-0.0395 upper=0.0 effort=40 velocity=0.333333333333333
- joint bio_gripper_g2_right_finger_joint: limit lower=0 upper=0.0395 effort=2.0 velocity=0.1 -> lower=0 upper=0.0395 effort=40 velocity=0.333333333333333

File: assets/urdf/xarm6/xarm6_1305_bio_gripper_g2_movable_visual.glb.urdf (robot description, URDF)
Before this commit: robot xarm6_1305_bio_gripper_g2_movable_visual.glb, 13 links, 12 joints
Links:
- link bio_gripper_g2_base_link: mass 0.38837 -> 0.765827; geometry collision mesh filename=../bio_gripper_g2/meshes/collision/bio_gripper_g2_base_link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; visual mesh filename=../bio_gripper_g2/meshes/visual/visual_glb/bio_gripper_g2_b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
- link bio_gripper_g2_left_finger: geometry collision mesh filename=../bio_gripper_g2/meshes/collision/bio_gripper_g2_left_fing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; collision mesh filename=../bio_gripper_g2/meshes/collision/bio_gripper_g2_left_fing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
- link bio_gripper_g2_right_finger: geometry collision mesh filename=../bio_gripper_g2/meshes/collision/bio_gripper_g2_right_fin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; collision mesh filename=../bio_gripper_g2/meshes/collision/bio_gripper_g2_right_fin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
Joints:
- joint bio_gripper_g2_left_finger_joint: limit lower=-0.0395 upper=0.0 effort=2.0 velocity=0.1 -> lower=-0.0395 upper=0.0 effort=40 velocity=0.333333333333333
- joint bio_gripper_g2_right_finger_joint: limit lower=0 upper=0.0395 effort=2.0 velocity=0.1 -> lower=0 upper=0.0395 effort=40 velocity=0.333333333333333

File: assets/urdf/xarm6/xarm6_1305_bio_gripper_g2_visual.glb.urdf (robot description, URDF)
Before this commit: robot xarm6_1305_bio_gripper_g2_visual.glb, 14 links, 13 joints
Links:
- link bio_gripper_g2_base_link: mass 0.38837 -> 0.765827; geometry collision mesh filename=../bio_gripper_g2/meshes/collision/bio_gripper_g2_base_link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
- link bio_gripper_g2_left_finger: geometry collision mesh filename=../bio_gripper_g2/meshes/collision/bio_gripper_g2_left_fing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; collision mesh filename=../bio_gripper_g2/meshes/collision/bio_gripper_g2_left_fing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
- link bio_gripper_g2_right_finger: geometry collision mesh filename=../bio_gripper_g2/meshes/collision/bio_gripper_g2_right_fin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; collision mesh filename=../bio_gripper_g2/meshes/collision/bio_gripper_g2_right_fin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
Joints:
- joint bio_gripper_g2_left_finger_joint: limit lower=-0.0395 upper=0.0 effort=2.0 velocity=0.1 -> lower=-0.0395 upper=0.0 effort=40 velocity=0.333333333333333
- joint bio_gripper_g2_right_finger_joint: limit lower=0 upper=0.0395 effort=2.0 velocity=0.1 -> lower=0 upper=0.0395 effort=40 velocity=0.333333333333333

File: assets/urdf/xarm7/xarm7_1305_bio_gripper_g2_movable_visual.glb.urdf (robot description, URDF)
Before this commit: robot xarm7_1305_bio_gripper_g2_movable_visual.glb, 13 links, 12 joints
Links:
- link bio_gripper_g2_base_link: mass 0.38837 -> 0.765827; geometry collision mesh filename=../bio_gripper_g2/meshes/collision/bio_gripper_g2_base_link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; visual mesh filename=../bio_gripper_g2/meshes/visual/visual_glb/bio_gripper_g2_b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
- link bio_gripper_g2_left_finger: geometry collision mesh filename=../bio_gripper_g2/meshes/collision/bio_gripper_g2_left_fing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; collision mesh filename=../bio_gripper_g2/meshes/collision/bio_gripper_g2_left_fing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
- link bio_gripper_g2_right_finger: geometry collision mesh filename=../bio_gripper_g2/meshes/collision/bio_gripper_g2_right_fin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; collision mesh filename=../bio_gripper_g2/meshes/collision/bio_gripper_g2_right_fin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
Joints:
- joint bio_gripper_g2_left_finger_joint: limit lower=-0.0395 upper=0.0 effort=2.0 velocity=0.1 -> lower=-0.0395 upper=0.0 effort=40 velocity=0.333333333333333
- joint bio_gripper_g2_right_finger_joint: limit lower=0 upper=0.0395 effort=2.0 velocity=0.1 -> lower=0 upper=0.0395 effort=40 velocity=0.333333333333333

File: assets/urdf/xarm7/xarm7_1305_bio_gripper_g2_visual.glb.urdf (robot description, URDF)
Before this commit: robot xarm7_1305_bio_gripper_g2_visual.glb, 14 links, 13 joints
Links:
- link bio_gripper_g2_base_link: mass 0.38837 -> 0.765827; geometry collision mesh filename=../bio_gripper_g2/meshes/collision/bio_gripper_g2_base_link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
- link bio_gripper_g2_left_finger: geometry collision mesh filename=../bio_gripper_g2/meshes/collision/bio_gripper_g2_left_fing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; collision mesh filename=../bio_gripper_g2/meshes/collision/bio_gripper_g2_left_fing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
- link bio_gripper_g2_right_finger: geometry collision mesh filename=../bio_gripper_g2/meshes/collision/bio_gripper_g2_right_fin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; collision mesh filename=../bio_gripper_g2/meshes/collision/bio_gripper_g2_right_fin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
Joints:
- joint bio_gripper_g2_left_finger_joint: limit lower=-0.0395 upper=0.0 effort=2.0 velocity=0.1 -> lower=-0.0395 upper=0.0 effort=40 velocity=0.333333333333333
- joint bio_gripper_g2_right_finger_joint: limit lower=0 upper=0.0395 effort=2.0 velocity=0.1 -> lower=0 upper=0.0395 effort=40 velocity=0.333333333333333
