Commit message: Release v0.2.8: Draco assets, TCP offset FK/IK, and project-check CI.
Co-authored-by: Cursor <cursoragent@cursor.com>

File: assets/urdf/bio_gripper_g2/bio_gripper_g2_movable_visual.urdf (robot description, URDF)
Before this commit: robot bio_gripper_g2_movable_visual, 5 links, 4 joints
Links:
- link bio_gripper_g2_base_link: geometry collision mesh filename=../bio_gripper_g2/meshes/visual/bio_gripper_g2_link_base.stl; visual mesh filename=../bio_gripper_g2/meshes/visual/visual_glb/bio_gripper_g2_b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
- link bio_gripper_g2_left_finger: geometry collision mesh filename=../bio_gripper_g2/meshes/visual/bio_gripper_g2_left_finger.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; visual mesh filename=../bio_gripper_g2/meshes/visual/visual_glb/bio_gripper_g2_l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
- link bio_gripper_g2_right_finger: geometry collision mesh filename=../bio_gripper_g2/meshes/visual/bio_gripper_g2_right_finger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; visual mesh filename=../bio_gripper_g2/meshes/visual/visual_glb/bio_gripper_g2_r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

File: assets/urdf/gripper_g2/gripper_g2_movable_visual.urdf (robot description, URDF)
Before this commit: robot gripper_g2_movable_visual, 9 links, 8 joints
Links:
- link xarm_gripper_base_link: geometry collision mesh filename=../gripper_g2/meshes/collision/base_link.stl; visual mesh filename=../gripper_g2/meshes/visual/visual_glb/base.glb

File: assets/urdf/uf850/uf850_bio_gripper_g2_movable_visual.glb.urdf (robot description, URDF)
Before this commit: robot uf850_bio_gripper_g2_movable_visual.glb, 12 links, 11 joints
Links:
- link bio_gripper_g2_base_link: geometry collision mesh filename=../bio_gripper_g2/meshes/visual/bio_gripper_g2_link_base.stl; visual mesh filename=../bio_gripper_g2/meshes/visual/visual_glb/bio_gripper_g2_b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
- link bio_gripper_g2_left_finger: geometry collision mesh filename=../bio_gripper_g2/meshes/visual/bio_gripper_g2_left_finger.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; visual mesh filename=../bio_gripper_g2/meshes/visual/visual_glb/bio_gripper_g2_l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
- link bio_gripper_g2_right_finger: geometry collision mesh filename=../bio_gripper_g2/meshes/visual/bio_gripper_g2_right_finger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; visual mesh filename=../bio_gripper_g2/meshes/visual/visual_glb/bio_gripper_g2_r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

File: assets/urdf/uf850/uf850_bio_gripper_g2_visual.glb.urdf (robot description, URDF)
Before this commit: robot uf850_bio_gripper_g2_visual.glb, 13 links, 12 joints
Links:
- link bio_gripper_g2_visual: geometry visual mesh filename=../bio_gripper_g2/meshes/visual/bio_gripper_g2_visual.glb

File: assets/urdf/uf850/uf850_g2_movable_visual.urdf (robot description, URDF)
Before this commit: robot uf850_g2_movable_visual, 16 links, 15 joints
Links:
- link xarm_gripper_base_link: geometry collision mesh filename=../gripper_g2/meshes/collision/base_link.stl; visual mesh filename=../gripper_g2/meshes/visual/visual_glb/base.glb

File: assets/urdf/uf850/uf850_g2_visual.urdf (robot description, URDF)
Before this commit: robot uf850_g2_visual, 17 links, 16 joints
Links:
- link gripper_g2_visual: geometry visual mesh filename=../gripper_g2/meshes/visual/gripper_g2_static.glb

File: assets/urdf/xarm5/xarm5_1305_bio_gripper_g2_movable_visual.glb.urdf (robot description, URDF)
Before this commit: robot xarm5_1305_bio_gripper_g2_movable_visual.glb, 11 links, 10 joints
Links:
- link bio_gripper_g2_base_link: geometry collision mesh filename=../bio_gripper_g2/meshes/visual/bio_gripper_g2_link_base.stl; visual mesh filename=../bio_gripper_g2/meshes/visual/visual_glb/bio_gripper_g2_b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
- link bio_gripper_g2_left_finger: geometry collision mesh filename=../bio_gripper_g2/meshes/visual/bio_gripper_g2_left_finger.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; visual mesh filename=../bio_gripper_g2/meshes/visual/visual_glb/bio_gripper_g2_l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
- link bio_gripper_g2_right_finger: geometry collision mesh filename=../bio_gripper_g2/meshes/visual/bio_gripper_g2_right_finger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; visual mesh filename=../bio_gripper_g2/meshes/visual/visual_glb/bio_gripper_g2_r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

File: assets/urdf/xarm5/xarm5_1305_bio_gripper_g2_visual.glb.urdf (robot description, URDF)
Before this commit: robot xarm5_1305_bio_gripper_g2_visual.glb, 12 links, 11 joints
Links:
- link bio_gripper_g2_visual: geometry visual mesh filename=../bio_gripper_g2/meshes/visual/bio_gripper_g2_visual.glb

File: assets/urdf/xarm5/xarm5_1305_g2_movable_visual.urdf (robot description, URDF)
Before this commit: robot xarm5_1305_g2_movable_visual, 15 links, 14 joints
Links:
- link xarm_gripper_base_link: geometry collision mesh filename=../gripper_g2/meshes/collision/base_link.stl; visual mesh filename=../gripper_g2/meshes/visual/visual_glb/base.glb

File: assets/urdf/xarm5/xarm5_1305_g2_visual.urdf (robot description, URDF)
Before this commit: robot xarm5_1305_g2_visual, 16 links, 15 joints
Links:
- link gripper_g2_visual: geometry visual mesh filename=../gripper_g2/meshes/visual/gripper_g2_static.glb

File: assets/urdf/xarm6/xarm6_1305_bio_gripper_g2_movable_visual.glb.urdf (robot description, URDF)
Before this commit: robot xarm6_1305_bio_gripper_g2_movable_visual.glb, 13 links, 12 joints
Links:
- link bio_gripper_g2_base_link: geometry collision mesh filename=../bio_gripper_g2/meshes/visual/bio_gripper_g2_link_base.stl; visual mesh filename=../bio_gripper_g2/meshes/visual/visual_glb/bio_gripper_g2_b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
- link bio_gripper_g2_left_finger: geometry collision mesh filename=../bio_gripper_g2/meshes/visual/bio_gripper_g2_left_finger.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; visual mesh filename=../bio_gripper_g2/meshes/visual/visual_glb/bio_gripper_g2_l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
- link bio_gripper_g2_right_finger: geometry collision mesh filename=../bio_gripper_g2/meshes/visual/bio_gripper_g2_right_finger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; visual mesh filename=../bio_gripper_g2/meshes/visual/visual_glb/bio_gripper_g2_r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

File: assets/urdf/xarm6/xarm6_1305_bio_gripper_g2_visual.glb.urdf (robot description, URDF)
Before this commit: robot xarm6_1305_bio_gripper_g2_visual.glb, 14 links, 13 joints
Links:
- link bio_gripper_g2_visual: geometry visual mesh filename=../bio_gripper_g2/meshes/visual/bio_gripper_g2_visual.glb

File: assets/urdf/xarm6/xarm6_1305_g2_movable_visual.urdf (robot description, URDF)
Before this commit: robot xarm6_1305_g2_movable_visual, 17 links, 16 joints
Links:
- link xarm_gripper_base_link: geometry collision mesh filename=../gripper_g2/meshes/collision/base_link.stl; visual mesh filename=../gripper_g2/meshes/visual/visual_glb/base.glb

File: assets/urdf/xarm6/xarm6_1305_g2_visual.urdf (robot description, URDF)
Before this commit: robot xarm6_1305_g2_visual, 18 links, 17 joints
Links:
- link gripper_g2_visual: geometry visual mesh filename=../gripper_g2/meshes/visual/gripper_g2_static.glb

File: assets/urdf/xarm7/xarm7_1305_bio_gripper_g2_movable_visual.glb.urdf (robot description, URDF)
Before this commit: robot xarm7_1305_bio_gripper_g2_movable_visual.glb, 13 links, 12 joints
Links:
- link bio_gripper_g2_base_link: geometry collision mesh filename=../bio_gripper_g2/meshes/visual/bio_gripper_g2_link_base.stl; visual mesh filename=../bio_gripper_g2/meshes/visual/visual_glb/bio_gripper_g2_b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
- link bio_gripper_g2_left_finger: geometry collision mesh filename=../bio_gripper_g2/meshes/visual/bio_gripper_g2_left_finger.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; visual mesh filename=../bio_gripper_g2/meshes/visual/visual_glb/bio_gripper_g2_l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
- link bio_gripper_g2_right_finger: geometry collision mesh filename=../bio_gripper_g2/meshes/visual/bio_gripper_g2_right_finger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; visual mesh filename=../bio_gripper_g2/meshes/visual/visual_glb/bio_gripper_g2_r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

File: assets/urdf/xarm7/xarm7_1305_bio_gripper_g2_visual.glb.urdf (robot description, URDF)
Before this commit: robot xarm7_1305_bio_gripper_g2_visual.glb, 14 links, 13 joints
Links:
- link bio_gripper_g2_visual: geometry visual mesh filename=../bio_gripper_g2/meshes/visual/bio_gripper_g2_visual.glb

File: assets/urdf/xarm7/xarm7_1305_g2_movable_visual.urdf (robot description, URDF)
Before this commit: robot xarm7_1305_g2_movable_visual, 17 links, 16 joints
Links:
- link xarm_gripper_base_link: geometry collision mesh filename=../gripper_g2/meshes/collision/base_link.stl; visual mesh filename=../gripper_g2/meshes/visual/visual_glb/base.glb

File: assets/urdf/xarm7/xarm7_1305_g2_visual.urdf (robot description, URDF)
Before this commit: robot xarm7_1305_g2_visual, 18 links, 17 joints
Links:
- link gripper_g2_visual: geometry visual mesh filename=../gripper_g2/meshes/visual/gripper_g2_static.glb
