Commit message: Release v0.2.7: task-oriented examples, packaging package, and Genesis 1.2.2.
Co-authored-by: Cursor <cursoragent@cursor.com>

File: assets/urdf/lite6/lite6_gripper_movable_visual.glb.urdf (robot description, URDF)
Before this commit: robot lite6_gripper_movable_visual.glb, 12 links, 11 joints
Links:
- link uflite_finger1: geometry collision box size=0.02 0.00425 0.01975; collision box size=0.02 0.0155 0.0095
- link uflite_finger2: geometry collision box size=0.02 0.00425 0.01975; collision box size=0.02 0.0155 0.0095

File: assets/urdf/lite6/lite6_gripper_reversed_movable_visual.glb.urdf (robot description, URDF)
Before this commit: robot lite6_gripper_reversed_movable_visual.glb, 12 links, 11 joints
Links:
- link uflite_finger1: geometry collision box size=0.02 0.00425 0.01975; collision box size=0.02 0.0155 0.0095
- link uflite_finger2: geometry collision box size=0.02 0.00425 0.01975; collision box size=0.02 0.0155 0.0095

File: assets/urdf/lite6/lite6_gripper_visual.glb.urdf (robot description, URDF)
Before this commit: robot lite6_gripper_visual.glb, 13 links, 12 joints
Links:
- link uflite_finger1: geometry collision box size=0.02 0.00425 0.01975; collision box size=0.02 0.0155 0.0095
- link uflite_finger2: geometry collision box size=0.02 0.00425 0.01975; collision box size=0.02 0.0155 0.0095

File: assets/urdf/lite6/lite6_with_gripper.urdf (robot description, URDF)
Before this commit: robot lite6_with_gripper, 12 links, 11 joints
Links:
- link uflite_finger1: geometry collision box size=0.02 0.00425 0.01975; collision box size=0.02 0.0155 0.0095
- link uflite_finger2: geometry collision box size=0.02 0.00425 0.01975; collision box size=0.02 0.0155 0.0095

File: assets/urdf/lite6_gripper/lite6_gripper.urdf (robot description, URDF)
Before this commit: robot lite6_gripper, 4 links, 4 joints
Links:
- link uflite_finger1: geometry collision box size=0.02 0.00425 0.01975; collision box size=0.02 0.0155 0.0095
- link uflite_finger2: geometry collision box size=0.02 0.00425 0.01975; collision box size=0.02 0.0155 0.0095

File: assets/urdf/lite6_gripper/lite6_gripper_movable_visual.urdf (robot description, URDF)
Before this commit: robot lite6_gripper_movable_visual, 5 links, 4 joints
Links:
- link uflite_finger1: geometry collision box size=0.02 0.00425 0.01975; collision box size=0.02 0.0155 0.0095
- link uflite_finger2: geometry collision box size=0.02 0.00425 0.01975; collision box size=0.02 0.0155 0.0095

File: assets/urdf/uf850/uf850_bio_gripper_g2_movable_visual.glb.urdf (robot description, URDF)
Before this commit: robot uf850_bio_gripper_g2_movable_visual.glb, 12 links, 11 joints
Joints:
- joint bio_gripper_g2_attach: origin xyz=0.024657 0.012975 -0.000386 rpy=0.00000000 0.00000000 0.47492066 -> xyz=0.024657 0 0 rpy=0 0 0

File: assets/urdf/uf850/uf850_bio_gripper_g2_visual.glb.urdf (robot description, URDF)
Before this commit: robot uf850_bio_gripper_g2_visual.glb, 13 links, 12 joints
Joints:
- joint bio_gripper_g2_attach: origin xyz=0.024657 0.012975 -0.000386 rpy=0.00000000 0.00000000 0.47492066 -> xyz=0.024657 0 0 rpy=0 0 0
- joint bio_gripper_g2_visual_fix: origin xyz=0.024657 0.012975 -0.000386 rpy=0.00000000 0.00000000 0.47492066 -> xyz=0.024657 0 0 rpy=0 0 0
