Commit message: Use official joint torque limits so PD hold saturates at the real output.
Retune Lite 6 direct-drive wrist friction and PD to those limits so J4 and J6 settle in the dynamics check.

Co-authored-by: Cursor <cursoragent@cursor.com>

File: assets/urdf/lite6/lite6.urdf (robot description, URDF)
Before this commit: robot gen, 8 links, 7 joints
Joints:
- joint joint1: limit lower=-6.283185307179586 upper=6.283185307179586 effort=50.0 velocity=3.14 -> lower=-6.283185307179586 upper=6.283185307179586 effort=81.6 velocity=3.14
- joint joint2: limit lower=-2.61799 upper=2.61799 effort=50.0 velocity=3.14 -> lower=-2.61799 upper=2.61799 effort=81.6 velocity=3.14
- joint joint3: limit lower=-0.061087 upper=5.235988 effort=32.0 velocity=3.14 -> lower=-0.061087 upper=5.235988 effort=30.6 velocity=3.14
- joint joint4: limit lower=-6.283185307179586 upper=6.283185307179586 effort=32.0 velocity=3.14 -> lower=-6.283185307179586 upper=6.283185307179586 effort=1.364505 velocity=3.14
- joint joint5: limit lower=-2.1642 upper=2.1642 effort=32.0 velocity=3.14 -> lower=-2.1642 upper=2.1642 effort=3.274812 velocity=3.14
- joint joint6: limit lower=-6.283185307179586 upper=6.283185307179586 effort=20.0 velocity=3.14 -> lower=-6.283185307179586 upper=6.283185307179586 effort=1.364505 velocity=3.14

File: assets/urdf/lite6/lite6_gripper_movable_visual.glb.urdf (robot description, URDF)
Before this commit: robot lite6_gripper_movable_visual.glb, 12 links, 11 joints
Joints:
- joint joint1: limit lower=-6.283185307179586 upper=6.283185307179586 effort=50.0 velocity=3.14 -> lower=-6.283185307179586 upper=6.283185307179586 effort=81.6 velocity=3.14
- joint joint2: limit lower=-2.61799 upper=2.61799 effort=50.0 velocity=3.14 -> lower=-2.61799 upper=2.61799 effort=81.6 velocity=3.14
- joint joint3: limit lower=-0.061087 upper=5.235988 effort=32.0 velocity=3.14 -> lower=-0.061087 upper=5.235988 effort=30.6 velocity=3.14
- joint joint4: limit lower=-6.283185307179586 upper=6.283185307179586 effort=32.0 velocity=3.14 -> lower=-6.283185307179586 upper=6.283185307179586 effort=1.364505 velocity=3.14
- joint joint5: limit lower=-2.1642 upper=2.1642 effort=32.0 velocity=3.14 -> lower=-2.1642 upper=2.1642 effort=3.274812 velocity=3.14
- joint joint6: limit lower=-6.283185307179586 upper=6.283185307179586 effort=20.0 velocity=3.14 -> lower=-6.283185307179586 upper=6.283185307179586 effort=1.364505 velocity=3.14

File: assets/urdf/lite6/lite6_gripper_reversed_movable_visual.glb.urdf (robot description, URDF)
Before this commit: robot lite6_gripper_reversed_movable_visual.glb, 12 links, 11 joints
Joints:
- joint joint1: limit lower=-6.283185307179586 upper=6.283185307179586 effort=50.0 velocity=3.14 -> lower=-6.283185307179586 upper=6.283185307179586 effort=81.6 velocity=3.14
- joint joint2: limit lower=-2.61799 upper=2.61799 effort=50.0 velocity=3.14 -> lower=-2.61799 upper=2.61799 effort=81.6 velocity=3.14
- joint joint3: limit lower=-0.061087 upper=5.235988 effort=32.0 velocity=3.14 -> lower=-0.061087 upper=5.235988 effort=30.6 velocity=3.14
- joint joint4: limit lower=-6.283185307179586 upper=6.283185307179586 effort=32.0 velocity=3.14 -> lower=-6.283185307179586 upper=6.283185307179586 effort=1.364505 velocity=3.14
- joint joint5: limit lower=-2.1642 upper=2.1642 effort=32.0 velocity=3.14 -> lower=-2.1642 upper=2.1642 effort=3.274812 velocity=3.14
- joint joint6: limit lower=-6.283185307179586 upper=6.283185307179586 effort=20.0 velocity=3.14 -> lower=-6.283185307179586 upper=6.283185307179586 effort=1.364505 velocity=3.14

File: assets/urdf/lite6/lite6_gripper_visual.glb.urdf (robot description, URDF)
Before this commit: robot lite6_gripper_visual.glb, 13 links, 12 joints
Joints:
- joint joint1: limit lower=-6.283185307179586 upper=6.283185307179586 effort=50.0 velocity=3.14 -> lower=-6.283185307179586 upper=6.283185307179586 effort=81.6 velocity=3.14
- joint joint2: limit lower=-2.61799 upper=2.61799 effort=50.0 velocity=3.14 -> lower=-2.61799 upper=2.61799 effort=81.6 velocity=3.14
- joint joint3: limit lower=-0.061087 upper=5.235988 effort=32.0 velocity=3.14 -> lower=-0.061087 upper=5.235988 effort=30.6 velocity=3.14
- joint joint4: limit lower=-6.283185307179586 upper=6.283185307179586 effort=32.0 velocity=3.14 -> lower=-6.283185307179586 upper=6.283185307179586 effort=1.364505 velocity=3.14
- joint joint5: limit lower=-2.1642 upper=2.1642 effort=32.0 velocity=3.14 -> lower=-2.1642 upper=2.1642 effort=3.274812 velocity=3.14
- joint joint6: limit lower=-6.283185307179586 upper=6.283185307179586 effort=20.0 velocity=3.14 -> lower=-6.283185307179586 upper=6.283185307179586 effort=1.364505 velocity=3.14

File: assets/urdf/lite6/lite6_vacuum_gripper_visual.glb.urdf (robot description, URDF)
Before this commit: robot lite6_vacuum_gripper_visual.glb, 9 links, 8 joints
Joints:
- joint joint1: limit lower=-6.283185307179586 upper=6.283185307179586 effort=50.0 velocity=3.14 -> lower=-6.283185307179586 upper=6.283185307179586 effort=81.6 velocity=3.14
- joint joint2: limit lower=-2.61799 upper=2.61799 effort=50.0 velocity=3.14 -> lower=-2.61799 upper=2.61799 effort=81.6 velocity=3.14
- joint joint3: limit lower=-0.061087 upper=5.235988 effort=32.0 velocity=3.14 -> lower=-0.061087 upper=5.235988 effort=30.6 velocity=3.14
- joint joint4: limit lower=-6.283185307179586 upper=6.283185307179586 effort=32.0 velocity=3.14 -> lower=-6.283185307179586 upper=6.283185307179586 effort=1.364505 velocity=3.14
- joint joint5: limit lower=-2.1642 upper=2.1642 effort=32.0 velocity=3.14 -> lower=-2.1642 upper=2.1642 effort=3.274812 velocity=3.14
- joint joint6: limit lower=-6.283185307179586 upper=6.283185307179586 effort=20.0 velocity=3.14 -> lower=-6.283185307179586 upper=6.283185307179586 effort=1.364505 velocity=3.14

File: assets/urdf/lite6/lite6_visual.glb.urdf (robot description, URDF)
Before this commit: robot gen, 8 links, 7 joints
Joints:
- joint joint1: limit lower=-6.283185307179586 upper=6.283185307179586 effort=50.0 velocity=3.14 -> lower=-6.283185307179586 upper=6.283185307179586 effort=81.6 velocity=3.14
- joint joint2: limit lower=-2.61799 upper=2.61799 effort=50.0 velocity=3.14 -> lower=-2.61799 upper=2.61799 effort=81.6 velocity=3.14
- joint joint3: limit lower=-0.061087 upper=5.235988 effort=32.0 velocity=3.14 -> lower=-0.061087 upper=5.235988 effort=30.6 velocity=3.14
- joint joint4: limit lower=-6.283185307179586 upper=6.283185307179586 effort=32.0 velocity=3.14 -> lower=-6.283185307179586 upper=6.283185307179586 effort=1.364505 velocity=3.14
- joint joint5: limit lower=-2.1642 upper=2.1642 effort=32.0 velocity=3.14 -> lower=-2.1642 upper=2.1642 effort=3.274812 velocity=3.14
- joint joint6: limit lower=-6.283185307179586 upper=6.283185307179586 effort=20.0 velocity=3.14 -> lower=-6.283185307179586 upper=6.283185307179586 effort=1.364505 velocity=3.14

File: assets/urdf/lite6/lite6_with_gripper.urdf (robot description, URDF)
Before this commit: robot lite6_with_gripper, 12 links, 11 joints
Joints:
- joint joint1: limit lower=-6.283185307179586 upper=6.283185307179586 effort=50.0 velocity=3.14 -> lower=-6.283185307179586 upper=6.283185307179586 effort=81.6 velocity=3.14
- joint joint2: limit lower=-2.61799 upper=2.61799 effort=50.0 velocity=3.14 -> lower=-2.61799 upper=2.61799 effort=81.6 velocity=3.14
- joint joint3: limit lower=-0.061087 upper=5.235988 effort=32.0 velocity=3.14 -> lower=-0.061087 upper=5.235988 effort=30.6 velocity=3.14
- joint joint4: limit lower=-6.283185307179586 upper=6.283185307179586 effort=32.0 velocity=3.14 -> lower=-6.283185307179586 upper=6.283185307179586 effort=1.364505 velocity=3.14
- joint joint5: limit lower=-2.1642 upper=2.1642 effort=32.0 velocity=3.14 -> lower=-2.1642 upper=2.1642 effort=3.274812 velocity=3.14
- joint joint6: limit lower=-6.283185307179586 upper=6.283185307179586 effort=20.0 velocity=3.14 -> lower=-6.283185307179586 upper=6.283185307179586 effort=1.364505 velocity=3.14

File: assets/urdf/lite6/lite6_with_vacuum_gripper.urdf (robot description, URDF)
Before this commit: robot lite6_with_vacuum_gripper, 10 links, 9 joints
Joints:
- joint joint1: limit lower=-6.283185307179586 upper=6.283185307179586 effort=50.0 velocity=3.14 -> lower=-6.283185307179586 upper=6.283185307179586 effort=81.6 velocity=3.14
- joint joint2: limit lower=-2.61799 upper=2.61799 effort=50.0 velocity=3.14 -> lower=-2.61799 upper=2.61799 effort=81.6 velocity=3.14
- joint joint3: limit lower=-0.061087 upper=5.235988 effort=32.0 velocity=3.14 -> lower=-0.061087 upper=5.235988 effort=30.6 velocity=3.14
- joint joint4: limit lower=-6.283185307179586 upper=6.283185307179586 effort=32.0 velocity=3.14 -> lower=-6.283185307179586 upper=6.283185307179586 effort=1.364505 velocity=3.14
- joint joint5: limit lower=-2.1642 upper=2.1642 effort=32.0 velocity=3.14 -> lower=-2.1642 upper=2.1642 effort=3.274812 velocity=3.14
- joint joint6: limit lower=-6.283185307179586 upper=6.283185307179586 effort=20.0 velocity=3.14 -> lower=-6.283185307179586 upper=6.283185307179586 effort=1.364505 velocity=3.14

File: assets/urdf/uf850/uf850.urdf (robot description, URDF)
Before this commit: robot gen, 8 links, 7 joints
Joints:
- joint joint1: limit lower=-6.283185307179586 upper=6.283185307179586 effort=200.0 velocity=3.14 -> lower=-6.283185307179586 upper=6.283185307179586 effort=382.5 velocity=3.14
- joint joint2: limit lower=-2.3038346 upper=2.3038346 effort=200.0 velocity=3.14 -> lower=-2.3038346 upper=2.3038346 effort=382.5 velocity=3.14
- joint joint3: limit lower=-4.2236968 upper=0.061087 effort=90.0 velocity=3.14 -> lower=-4.2236968 upper=0.061087 effort=243.525 velocity=3.14
- joint joint4: limit lower=-6.283185307179586 upper=6.283185307179586 effort=68.0 velocity=3.14 -> lower=-6.283185307179586 upper=6.283185307179586 effort=117.3 velocity=3.14
- joint joint5: limit lower=-2.1642 upper=2.1642 effort=19.0 velocity=3.14 -> lower=-2.1642 upper=2.1642 effort=38.25 velocity=3.14
- joint joint6: limit lower=-6.283185307179586 upper=6.283185307179586 effort=19.0 velocity=3.14 -> lower=-6.283185307179586 upper=6.283185307179586 effort=38.25 velocity=3.14

File: assets/urdf/uf850/uf850_bio_gripper_g2_movable_visual.glb.urdf (robot description, URDF)
Before this commit: robot uf850_bio_gripper_g2_movable_visual.glb, 12 links, 11 joints
Joints:
- joint joint1: limit lower=-6.283185307179586 upper=6.283185307179586 effort=200.0 velocity=3.14 -> lower=-6.283185307179586 upper=6.283185307179586 effort=382.5 velocity=3.14
- joint joint2: limit lower=-2.3038346 upper=2.3038346 effort=200.0 velocity=3.14 -> lower=-2.3038346 upper=2.3038346 effort=382.5 velocity=3.14
- joint joint3: limit lower=-4.2236968 upper=0.061087 effort=90.0 velocity=3.14 -> lower=-4.2236968 upper=0.061087 effort=243.525 velocity=3.14
- joint joint4: limit lower=-6.283185307179586 upper=6.283185307179586 effort=68.0 velocity=3.14 -> lower=-6.283185307179586 upper=6.283185307179586 effort=117.3 velocity=3.14
- joint joint5: limit lower=-2.1642 upper=2.1642 effort=19.0 velocity=3.14 -> lower=-2.1642 upper=2.1642 effort=38.25 velocity=3.14
- joint joint6: limit lower=-6.283185307179586 upper=6.283185307179586 effort=19.0 velocity=3.14 -> lower=-6.283185307179586 upper=6.283185307179586 effort=38.25 velocity=3.14

File: assets/urdf/uf850/uf850_bio_gripper_g2_visual.glb.urdf (robot description, URDF)
Before this commit: robot uf850_bio_gripper_g2_visual.glb, 13 links, 12 joints
Joints:
- joint joint1: limit lower=-6.283185307179586 upper=6.283185307179586 effort=200.0 velocity=3.14 -> lower=-6.283185307179586 upper=6.283185307179586 effort=382.5 velocity=3.14
- joint joint2: limit lower=-2.3038346 upper=2.3038346 effort=200.0 velocity=3.14 -> lower=-2.3038346 upper=2.3038346 effort=382.5 velocity=3.14
- joint joint3: limit lower=-4.2236968 upper=0.061087 effort=90.0 velocity=3.14 -> lower=-4.2236968 upper=0.061087 effort=243.525 velocity=3.14
- joint joint4: limit lower=-6.283185307179586 upper=6.283185307179586 effort=68.0 velocity=3.14 -> lower=-6.283185307179586 upper=6.283185307179586 effort=117.3 velocity=3.14
- joint joint5: limit lower=-2.1642 upper=2.1642 effort=19.0 velocity=3.14 -> lower=-2.1642 upper=2.1642 effort=38.25 velocity=3.14
- joint joint6: limit lower=-6.283185307179586 upper=6.283185307179586 effort=19.0 velocity=3.14 -> lower=-6.283185307179586 upper=6.283185307179586 effort=38.25 velocity=3.14

File: assets/urdf/uf850/uf850_g2_movable_visual.urdf (robot description, URDF)
Before this commit: robot uf850_g2_movable_visual, 16 links, 15 joints
Joints:
- joint joint1: limit lower=-6.283185307179586 upper=6.283185307179586 effort=200.0 velocity=3.14 -> lower=-6.283185307179586 upper=6.283185307179586 effort=382.5 velocity=3.14
- joint joint2: limit lower=-2.3038346 upper=2.3038346 effort=200.0 velocity=3.14 -> lower=-2.3038346 upper=2.3038346 effort=382.5 velocity=3.14
- joint joint3: limit lower=-4.2236968 upper=0.061087 effort=90.0 velocity=3.14 -> lower=-4.2236968 upper=0.061087 effort=243.525 velocity=3.14
- joint joint4: limit lower=-6.283185307179586 upper=6.283185307179586 effort=68.0 velocity=3.14 -> lower=-6.283185307179586 upper=6.283185307179586 effort=117.3 velocity=3.14
- joint joint5: limit lower=-2.1642 upper=2.1642 effort=19.0 velocity=3.14 -> lower=-2.1642 upper=2.1642 effort=38.25 velocity=3.14
- joint joint6: limit lower=-6.283185307179586 upper=6.283185307179586 effort=19.0 velocity=3.14 -> lower=-6.283185307179586 upper=6.283185307179586 effort=38.25 velocity=3.14

File: assets/urdf/uf850/uf850_g2_visual.urdf (robot description, URDF)
Before this commit: robot uf850_g2_visual, 17 links, 16 joints
Joints:
- joint joint1: limit lower=-6.283185307179586 upper=6.283185307179586 effort=200.0 velocity=3.14 -> lower=-6.283185307179586 upper=6.283185307179586 effort=382.5 velocity=3.14
- joint joint2: limit lower=-2.3038346 upper=2.3038346 effort=200.0 velocity=3.14 -> lower=-2.3038346 upper=2.3038346 effort=382.5 velocity=3.14
- joint joint3: limit lower=-4.2236968 upper=0.061087 effort=90.0 velocity=3.14 -> lower=-4.2236968 upper=0.061087 effort=243.525 velocity=3.14
- joint joint4: limit lower=-6.283185307179586 upper=6.283185307179586 effort=68.0 velocity=3.14 -> lower=-6.283185307179586 upper=6.283185307179586 effort=117.3 velocity=3.14
- joint joint5: limit lower=-2.1642 upper=2.1642 effort=19.0 velocity=3.14 -> lower=-2.1642 upper=2.1642 effort=38.25 velocity=3.14
- joint joint6: limit lower=-6.283185307179586 upper=6.283185307179586 effort=19.0 velocity=3.14 -> lower=-6.283185307179586 upper=6.283185307179586 effort=38.25 velocity=3.14

File: assets/urdf/uf850/uf850_visual.glb.urdf (robot description, URDF)
Before this commit: robot gen, 8 links, 7 joints
Joints:
- joint joint1: limit lower=-6.283185307179586 upper=6.283185307179586 effort=200.0 velocity=3.14 -> lower=-6.283185307179586 upper=6.283185307179586 effort=382.5 velocity=3.14
- joint joint2: limit lower=-2.3038346 upper=2.3038346 effort=200.0 velocity=3.14 -> lower=-2.3038346 upper=2.3038346 effort=382.5 velocity=3.14
- joint joint3: limit lower=-4.2236968 upper=0.061087 effort=90.0 velocity=3.14 -> lower=-4.2236968 upper=0.061087 effort=243.525 velocity=3.14
- joint joint4: limit lower=-6.283185307179586 upper=6.283185307179586 effort=68.0 velocity=3.14 -> lower=-6.283185307179586 upper=6.283185307179586 effort=117.3 velocity=3.14
- joint joint5: limit lower=-2.1642 upper=2.1642 effort=19.0 velocity=3.14 -> lower=-2.1642 upper=2.1642 effort=38.25 velocity=3.14
- joint joint6: limit lower=-6.283185307179586 upper=6.283185307179586 effort=19.0 velocity=3.14 -> lower=-6.283185307179586 upper=6.283185307179586 effort=38.25 velocity=3.14

File: assets/urdf/xarm5/xarm5_1305.urdf (robot description, URDF)
Before this commit: robot gen, 7 links, 6 joints
Joints:
- joint joint1: limit lower=-6.283185307179586 upper=6.283185307179586 effort=50 velocity=3.14 -> lower=-6.283185307179586 upper=6.283185307179586 effort=179.4445 velocity=3.14
- joint joint2: limit lower=-2.059 upper=2.0944 effort=50 velocity=3.14 -> lower=-2.059 upper=2.0944 effort=179.4445 velocity=3.14
- joint joint3: limit lower=-3.927 upper=0.19198 effort=30 velocity=3.14 -> lower=-3.927 upper=0.19198 effort=92.0 velocity=3.14
- joint joint4: limit lower=-1.69297 upper=3.141592653589793 effort=20 velocity=3.14 -> lower=-1.69297 upper=3.141592653589793 effort=30.6 velocity=3.14
- joint joint5: limit lower=-6.283185307179586 upper=6.283185307179586 effort=20 velocity=3.14 -> lower=-6.283185307179586 upper=6.283185307179586 effort=30.6 velocity=3.14

File: assets/urdf/xarm5/xarm5_1305_bio_gripper_g2_movable_visual.glb.urdf (robot description, URDF)
Before this commit: robot xarm5_1305_bio_gripper_g2_movable_visual.glb, 11 links, 10 joints
Joints:
- joint joint1: limit lower=-6.283185307179586 upper=6.283185307179586 effort=50 velocity=3.14 -> lower=-6.283185307179586 upper=6.283185307179586 effort=179.4445 velocity=3.14
- joint joint2: limit lower=-2.059 upper=2.0944 effort=50 velocity=3.14 -> lower=-2.059 upper=2.0944 effort=179.4445 velocity=3.14
- joint joint3: limit lower=-3.927 upper=0.19198 effort=30 velocity=3.14 -> lower=-3.927 upper=0.19198 effort=92.0 velocity=3.14
- joint joint4: limit lower=-1.69297 upper=3.141592653589793 effort=20 velocity=3.14 -> lower=-1.69297 upper=3.141592653589793 effort=30.6 velocity=3.14
- joint joint5: limit lower=-6.283185307179586 upper=6.283185307179586 effort=20 velocity=3.14 -> lower=-6.283185307179586 upper=6.283185307179586 effort=30.6 velocity=3.14

File: assets/urdf/xarm5/xarm5_1305_bio_gripper_g2_visual.glb.urdf (robot description, URDF)
Before this commit: robot xarm5_1305_bio_gripper_g2_visual.glb, 12 links, 11 joints
Joints:
- joint joint1: limit lower=-6.283185307179586 upper=6.283185307179586 effort=50 velocity=3.14 -> lower=-6.283185307179586 upper=6.283185307179586 effort=179.4445 velocity=3.14
- joint joint2: limit lower=-2.059 upper=2.0944 effort=50 velocity=3.14 -> lower=-2.059 upper=2.0944 effort=179.4445 velocity=3.14
- joint joint3: limit lower=-3.927 upper=0.19198 effort=30 velocity=3.14 -> lower=-3.927 upper=0.19198 effort=92.0 velocity=3.14
- joint joint4: limit lower=-1.69297 upper=3.141592653589793 effort=20 velocity=3.14 -> lower=-1.69297 upper=3.141592653589793 effort=30.6 velocity=3.14
- joint joint5: limit lower=-6.283185307179586 upper=6.283185307179586 effort=20 velocity=3.14 -> lower=-6.283185307179586 upper=6.283185307179586 effort=30.6 velocity=3.14

File: assets/urdf/xarm5/xarm5_1305_g2_movable_visual.urdf (robot description, URDF)
Before this commit: robot xarm5_1305_g2_movable_visual, 15 links, 14 joints
Joints:
- joint joint1: limit lower=-6.283185307179586 upper=6.283185307179586 effort=50 velocity=3.14 -> lower=-6.283185307179586 upper=6.283185307179586 effort=179.4445 velocity=3.14
- joint joint2: limit lower=-2.059 upper=2.0944 effort=50 velocity=3.14 -> lower=-2.059 upper=2.0944 effort=179.4445 velocity=3.14
- joint joint3: limit lower=-3.927 upper=0.19198 effort=30 velocity=3.14 -> lower=-3.927 upper=0.19198 effort=92.0 velocity=3.14
- joint joint4: limit lower=-1.69297 upper=3.141592653589793 effort=20 velocity=3.14 -> lower=-1.69297 upper=3.141592653589793 effort=30.6 velocity=3.14
- joint joint5: limit lower=-6.283185307179586 upper=6.283185307179586 effort=20 velocity=3.14 -> lower=-6.283185307179586 upper=6.283185307179586 effort=30.6 velocity=3.14

File: assets/urdf/xarm5/xarm5_1305_g2_visual.urdf (robot description, URDF)
Before this commit: robot xarm5_1305_g2_visual, 16 links, 15 joints
Joints:
- joint joint1: limit lower=-6.283185307179586 upper=6.283185307179586 effort=50 velocity=3.14 -> lower=-6.283185307179586 upper=6.283185307179586 effort=179.4445 velocity=3.14
- joint joint2: limit lower=-2.059 upper=2.0944 effort=50 velocity=3.14 -> lower=-2.059 upper=2.0944 effort=179.4445 velocity=3.14
- joint joint3: limit lower=-3.927 upper=0.19198 effort=30 velocity=3.14 -> lower=-3.927 upper=0.19198 effort=92.0 velocity=3.14
- joint joint4: limit lower=-1.69297 upper=3.141592653589793 effort=20 velocity=3.14 -> lower=-1.69297 upper=3.141592653589793 effort=30.6 velocity=3.14
- joint joint5: limit lower=-6.283185307179586 upper=6.283185307179586 effort=20 velocity=3.14 -> lower=-6.283185307179586 upper=6.283185307179586 effort=30.6 velocity=3.14

File: assets/urdf/xarm5/xarm5_1305_visual.glb.urdf (robot description, URDF)
Before this commit: robot gen, 7 links, 6 joints
Joints:
- joint joint1: limit lower=-6.283185307179586 upper=6.283185307179586 effort=50 velocity=3.14 -> lower=-6.283185307179586 upper=6.283185307179586 effort=179.4445 velocity=3.14
- joint joint2: limit lower=-2.059 upper=2.0944 effort=50 velocity=3.14 -> lower=-2.059 upper=2.0944 effort=179.4445 velocity=3.14
- joint joint3: limit lower=-3.927 upper=0.19198 effort=30 velocity=3.14 -> lower=-3.927 upper=0.19198 effort=92.0 velocity=3.14
- joint joint4: limit lower=-1.69297 upper=3.141592653589793 effort=20 velocity=3.14 -> lower=-1.69297 upper=3.141592653589793 effort=30.6 velocity=3.14
- joint joint5: limit lower=-6.283185307179586 upper=6.283185307179586 effort=20 velocity=3.14 -> lower=-6.283185307179586 upper=6.283185307179586 effort=30.6 velocity=3.14
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