Commit message: Update arm collision meshes with selective convex hulls across 5 robots

File: assets/urdf/lite6/lite6.urdf (robot description, URDF)
Before this commit: robot gen, 8 links, 7 joints
Links:
- link link1: geometry collision mesh filename=meshes/lite6/collision/lite6_link1_col_00.stl; collision mesh filename=meshes/lite6/collision/lite6_link1_col_01.stl
- link link2: geometry collision mesh filename=meshes/lite6/collision/lite6_link2_col_00.stl; collision mesh filename=meshes/lite6/collision/lite6_link2_col_01.stl
- link link3: geometry collision mesh filename=meshes/lite6/collision/lite6_link3_col_00.stl; collision mesh filename=meshes/lite6/collision/lite6_link3_col_01.stl
- link link4: geometry collision mesh filename=meshes/lite6/collision/lite6_link4_col_00.stl; collision mesh filename=meshes/lite6/collision/lite6_link4_col_01.stl
- link link5: geometry collision mesh filename=meshes/lite6/collision/lite6_link5_col_00.stl; visual mesh filename=meshes/lite6/visual/link5.stl
- link link6: geometry collision mesh filename=meshes/lite6/collision/lite6_link6_col_00.stl; visual mesh filename=meshes/lite6/visual/link6.stl
- link link_base: geometry collision mesh filename=meshes/lite6/collision/lite6_link_base_col_00.stl; collision mesh filename=meshes/lite6/collision/lite6_link_base_col_01.stl

File: assets/urdf/lite6/lite6_gripper_movable_visual.glb.urdf (robot description, URDF)
Before this commit: robot lite6_gripper_movable_visual.glb, 12 links, 11 joints
Links:
- link link1: geometry collision mesh filename=meshes/lite6/collision/lite6_link1_col_00.stl; collision mesh filename=meshes/lite6/collision/lite6_link1_col_01.stl
- link link2: geometry collision mesh filename=meshes/lite6/collision/lite6_link2_col_00.stl; collision mesh filename=meshes/lite6/collision/lite6_link2_col_01.stl
- link link3: geometry collision mesh filename=meshes/lite6/collision/lite6_link3_col_00.stl; collision mesh filename=meshes/lite6/collision/lite6_link3_col_01.stl
- link link4: geometry collision mesh filename=meshes/lite6/collision/lite6_link4_col_00.stl; collision mesh filename=meshes/lite6/collision/lite6_link4_col_01.stl
- link link5: geometry collision mesh filename=meshes/lite6/collision/lite6_link5_col_00.stl; visual mesh filename=meshes/lite6/visual_glb/link5.glb
- link link6: geometry collision mesh filename=meshes/lite6/collision/lite6_link6_col_00.stl; visual mesh filename=meshes/lite6/visual_glb/link6.glb
- link link_base: geometry collision mesh filename=meshes/lite6/collision/lite6_link_base_col_00.stl; collision mesh filename=meshes/lite6/collision/lite6_link_base_col_01.stl

File: assets/urdf/lite6/lite6_gripper_reversed_movable_visual.glb.urdf (robot description, URDF)
Before this commit: robot lite6_gripper_reversed_movable_visual.glb, 12 links, 11 joints
Links:
- link link1: geometry collision mesh filename=meshes/lite6/collision/lite6_link1_col_00.stl; collision mesh filename=meshes/lite6/collision/lite6_link1_col_01.stl
- link link2: geometry collision mesh filename=meshes/lite6/collision/lite6_link2_col_00.stl; collision mesh filename=meshes/lite6/collision/lite6_link2_col_01.stl
- link link3: geometry collision mesh filename=meshes/lite6/collision/lite6_link3_col_00.stl; collision mesh filename=meshes/lite6/collision/lite6_link3_col_01.stl
- link link4: geometry collision mesh filename=meshes/lite6/collision/lite6_link4_col_00.stl; collision mesh filename=meshes/lite6/collision/lite6_link4_col_01.stl
- link link5: geometry collision mesh filename=meshes/lite6/collision/lite6_link5_col_00.stl; visual mesh filename=meshes/lite6/visual_glb/link5.glb
- link link6: geometry collision mesh filename=meshes/lite6/collision/lite6_link6_col_00.stl; visual mesh filename=meshes/lite6/visual_glb/link6.glb
- link link_base: geometry collision mesh filename=meshes/lite6/collision/lite6_link_base_col_00.stl; collision mesh filename=meshes/lite6/collision/lite6_link_base_col_01.stl

File: assets/urdf/lite6/lite6_gripper_visual.glb.urdf (robot description, URDF)
Before this commit: robot lite6_gripper_visual.glb, 13 links, 12 joints
Links:
- link link1: geometry collision mesh filename=meshes/lite6/collision/lite6_link1_col_00.stl; collision mesh filename=meshes/lite6/collision/lite6_link1_col_01.stl
- link link2: geometry collision mesh filename=meshes/lite6/collision/lite6_link2_col_00.stl; collision mesh filename=meshes/lite6/collision/lite6_link2_col_01.stl
- link link3: geometry collision mesh filename=meshes/lite6/collision/lite6_link3_col_00.stl; collision mesh filename=meshes/lite6/collision/lite6_link3_col_01.stl
- link link4: geometry collision mesh filename=meshes/lite6/collision/lite6_link4_col_00.stl; collision mesh filename=meshes/lite6/collision/lite6_link4_col_01.stl
- link link5: geometry collision mesh filename=meshes/lite6/collision/lite6_link5_col_00.stl; visual mesh filename=meshes/lite6/visual_glb/link5.glb
- link link6: geometry collision mesh filename=meshes/lite6/collision/lite6_link6_col_00.stl; visual mesh filename=meshes/lite6/visual_glb/link6.glb
- link link_base: geometry collision mesh filename=meshes/lite6/collision/lite6_link_base_col_00.stl; collision mesh filename=meshes/lite6/collision/lite6_link_base_col_01.stl

File: assets/urdf/lite6/lite6_vacuum_gripper_visual.glb.urdf (robot description, URDF)
Before this commit: robot lite6_vacuum_gripper_visual.glb, 9 links, 8 joints
Links:
- link link1: geometry collision mesh filename=meshes/lite6/collision/lite6_link1_col_00.stl; collision mesh filename=meshes/lite6/collision/lite6_link1_col_01.stl
- link link2: geometry collision mesh filename=meshes/lite6/collision/lite6_link2_col_00.stl; collision mesh filename=meshes/lite6/collision/lite6_link2_col_01.stl
- link link3: geometry collision mesh filename=meshes/lite6/collision/lite6_link3_col_00.stl; collision mesh filename=meshes/lite6/collision/lite6_link3_col_01.stl
- link link4: geometry collision mesh filename=meshes/lite6/collision/lite6_link4_col_00.stl; collision mesh filename=meshes/lite6/collision/lite6_link4_col_01.stl
- link link5: geometry collision mesh filename=meshes/lite6/collision/lite6_link5_col_00.stl; visual mesh filename=meshes/lite6/visual_glb/link5.glb
- link link6: geometry collision mesh filename=meshes/lite6/collision/lite6_link6_col_00.stl; visual mesh filename=meshes/lite6/visual_glb/link6.glb
- link link_base: geometry collision mesh filename=meshes/lite6/collision/lite6_link_base_col_00.stl; collision mesh filename=meshes/lite6/collision/lite6_link_base_col_01.stl

File: assets/urdf/lite6/lite6_visual.glb.urdf (robot description, URDF)
Before this commit: robot gen, 8 links, 7 joints
Links:
- link link1: geometry collision mesh filename=meshes/lite6/collision/lite6_link1_col_00.stl; collision mesh filename=meshes/lite6/collision/lite6_link1_col_01.stl
- link link2: geometry collision mesh filename=meshes/lite6/collision/lite6_link2_col_00.stl; collision mesh filename=meshes/lite6/collision/lite6_link2_col_01.stl
- link link3: geometry collision mesh filename=meshes/lite6/collision/lite6_link3_col_00.stl; collision mesh filename=meshes/lite6/collision/lite6_link3_col_01.stl
- link link4: geometry collision mesh filename=meshes/lite6/collision/lite6_link4_col_00.stl; collision mesh filename=meshes/lite6/collision/lite6_link4_col_01.stl
- link link5: geometry collision mesh filename=meshes/lite6/collision/lite6_link5_col_00.stl; visual mesh filename=meshes/lite6/visual_glb/link5.glb
- link link6: geometry collision mesh filename=meshes/lite6/collision/lite6_link6_col_00.stl; visual mesh filename=meshes/lite6/visual_glb/link6.glb
- link link_base: geometry collision mesh filename=meshes/lite6/collision/lite6_link_base_col_00.stl; collision mesh filename=meshes/lite6/collision/lite6_link_base_col_01.stl

File: assets/urdf/lite6/lite6_with_gripper.urdf (robot description, URDF)
Before this commit: robot lite6_with_gripper, 12 links, 11 joints
Links:
- link link1: geometry collision mesh filename=meshes/lite6/collision/lite6_link1_col_00.stl; collision mesh filename=meshes/lite6/collision/lite6_link1_col_01.stl
- link link2: geometry collision mesh filename=meshes/lite6/collision/lite6_link2_col_00.stl; collision mesh filename=meshes/lite6/collision/lite6_link2_col_01.stl
- link link3: geometry collision mesh filename=meshes/lite6/collision/lite6_link3_col_00.stl; collision mesh filename=meshes/lite6/collision/lite6_link3_col_01.stl
- link link4: geometry collision mesh filename=meshes/lite6/collision/lite6_link4_col_00.stl; collision mesh filename=meshes/lite6/collision/lite6_link4_col_01.stl
- link link5: geometry collision mesh filename=meshes/lite6/collision/lite6_link5_col_00.stl; visual mesh filename=meshes/lite6/visual/link5.stl
- link link6: geometry collision mesh filename=meshes/lite6/collision/lite6_link6_col_00.stl; visual mesh filename=meshes/lite6/visual/link6.stl
- link link_base: geometry collision mesh filename=meshes/lite6/collision/lite6_link_base_col_00.stl; collision mesh filename=meshes/lite6/collision/lite6_link_base_col_01.stl

File: assets/urdf/lite6/lite6_with_vacuum_gripper.urdf (robot description, URDF)
Before this commit: robot lite6_with_vacuum_gripper, 10 links, 9 joints
Links:
- link link1: geometry collision mesh filename=meshes/lite6/collision/lite6_link1_col_00.stl; collision mesh filename=meshes/lite6/collision/lite6_link1_col_01.stl
- link link2: geometry collision mesh filename=meshes/lite6/collision/lite6_link2_col_00.stl; collision mesh filename=meshes/lite6/collision/lite6_link2_col_01.stl
- link link3: geometry collision mesh filename=meshes/lite6/collision/lite6_link3_col_00.stl; collision mesh filename=meshes/lite6/collision/lite6_link3_col_01.stl
- link link4: geometry collision mesh filename=meshes/lite6/collision/lite6_link4_col_00.stl; collision mesh filename=meshes/lite6/collision/lite6_link4_col_01.stl
- link link5: geometry collision mesh filename=meshes/lite6/collision/lite6_link5_col_00.stl; visual mesh filename=meshes/lite6/visual/link5.stl
- link link6: geometry collision mesh filename=meshes/lite6/collision/lite6_link6_col_00.stl; visual mesh filename=meshes/lite6/visual/link6.stl
- link link_base: geometry collision mesh filename=meshes/lite6/collision/lite6_link_base_col_00.stl; collision mesh filename=meshes/lite6/collision/lite6_link_base_col_01.stl

File: assets/urdf/uf850/uf850.urdf (robot description, URDF)
Before this commit: robot gen, 8 links, 7 joints
Links:
- link link1: geometry collision mesh filename=meshes/uf850/collision/uf850_link1_col_00.stl; collision mesh filename=meshes/uf850/collision/uf850_link1_col_01.stl
- link link2: geometry collision mesh filename=meshes/uf850/collision/uf850_link2_col_00.stl; collision mesh filename=meshes/uf850/collision/uf850_link2_col_01.stl
- link link3: geometry collision mesh filename=meshes/uf850/collision/uf850_link3_col_00.stl; collision mesh filename=meshes/uf850/collision/uf850_link3_col_01.stl
- link link4: geometry collision mesh filename=meshes/uf850/collision/uf850_link4_col_00.stl; collision mesh filename=meshes/uf850/collision/uf850_link4_col_01.stl
- link link5: geometry collision mesh filename=meshes/uf850/collision/uf850_link5_col_00.stl; collision mesh filename=meshes/uf850/collision/uf850_link5_col_01.stl
- link link6: geometry collision mesh filename=meshes/uf850/collision/uf850_link6_col_00.stl; visual mesh filename=meshes/uf850/visual/link6.stl
- link link_base: geometry collision mesh filename=meshes/uf850/collision/uf850_link_base_col_00.stl; collision mesh filename=meshes/uf850/collision/uf850_link_base_col_01.stl

File: assets/urdf/uf850/uf850_bio_gripper_g2_movable_visual.glb.urdf (robot description, URDF)
Before this commit: robot uf850_bio_gripper_g2_movable_visual.glb, 12 links, 11 joints
Links:
- link link1: geometry collision mesh filename=meshes/uf850/collision/uf850_link1_col_00.stl; collision mesh filename=meshes/uf850/collision/uf850_link1_col_01.stl
- link link2: geometry collision mesh filename=meshes/uf850/collision/uf850_link2_col_00.stl; collision mesh filename=meshes/uf850/collision/uf850_link2_col_01.stl
- link link3: geometry collision mesh filename=meshes/uf850/collision/uf850_link3_col_00.stl; collision mesh filename=meshes/uf850/collision/uf850_link3_col_01.stl
- link link4: geometry collision mesh filename=meshes/uf850/collision/uf850_link4_col_00.stl; collision mesh filename=meshes/uf850/collision/uf850_link4_col_01.stl
- link link5: geometry collision mesh filename=meshes/uf850/collision/uf850_link5_col_00.stl; collision mesh filename=meshes/uf850/collision/uf850_link5_col_01.stl
- link link6: geometry collision mesh filename=meshes/uf850/collision/uf850_link6_col_00.stl; visual mesh filename=meshes/uf850/visual_glb/link6.glb
- link link_base: geometry collision mesh filename=meshes/uf850/collision/uf850_link_base_col_00.stl; collision mesh filename=meshes/uf850/collision/uf850_link_base_col_01.stl

File: assets/urdf/uf850/uf850_bio_gripper_g2_visual.glb.urdf (robot description, URDF)
Before this commit: robot uf850_bio_gripper_g2_visual.glb, 13 links, 12 joints
Links:
- link link1: geometry collision mesh filename=meshes/uf850/collision/uf850_link1_col_00.stl; collision mesh filename=meshes/uf850/collision/uf850_link1_col_01.stl
- link link2: geometry collision mesh filename=meshes/uf850/collision/uf850_link2_col_00.stl; collision mesh filename=meshes/uf850/collision/uf850_link2_col_01.stl
- link link3: geometry collision mesh filename=meshes/uf850/collision/uf850_link3_col_00.stl; collision mesh filename=meshes/uf850/collision/uf850_link3_col_01.stl
- link link4: geometry collision mesh filename=meshes/uf850/collision/uf850_link4_col_00.stl; collision mesh filename=meshes/uf850/collision/uf850_link4_col_01.stl
- link link5: geometry collision mesh filename=meshes/uf850/collision/uf850_link5_col_00.stl; collision mesh filename=meshes/uf850/collision/uf850_link5_col_01.stl
- link link6: geometry collision mesh filename=meshes/uf850/collision/uf850_link6_col_00.stl; visual mesh filename=meshes/uf850/visual_glb/link6.glb
- link link_base: geometry collision mesh filename=meshes/uf850/collision/uf850_link_base_col_00.stl; collision mesh filename=meshes/uf850/collision/uf850_link_base_col_01.stl

File: assets/urdf/uf850/uf850_g2_movable_visual.urdf (robot description, URDF)
Before this commit: robot uf850_g2_movable_visual, 16 links, 15 joints
Links:
- link link1: geometry collision mesh filename=meshes/uf850/collision/uf850_link1_col_00.stl; collision mesh filename=meshes/uf850/collision/uf850_link1_col_01.stl
- link link2: geometry collision mesh filename=meshes/uf850/collision/uf850_link2_col_00.stl; collision mesh filename=meshes/uf850/collision/uf850_link2_col_01.stl
- link link3: geometry collision mesh filename=meshes/uf850/collision/uf850_link3_col_00.stl; collision mesh filename=meshes/uf850/collision/uf850_link3_col_01.stl
- link link4: geometry collision mesh filename=meshes/uf850/collision/uf850_link4_col_00.stl; collision mesh filename=meshes/uf850/collision/uf850_link4_col_01.stl
- link link5: geometry collision mesh filename=meshes/uf850/collision/uf850_link5_col_00.stl; collision mesh filename=meshes/uf850/collision/uf850_link5_col_01.stl
- link link6: geometry collision mesh filename=meshes/uf850/collision/uf850_link6_col_00.stl; visual mesh filename=meshes/uf850/visual_glb/link6.glb
- link link_base: geometry collision mesh filename=meshes/uf850/collision/uf850_link_base_col_00.stl; collision mesh filename=meshes/uf850/collision/uf850_link_base_col_01.stl

File: assets/urdf/uf850/uf850_g2_visual.urdf (robot description, URDF)
Before this commit: robot uf850_g2_visual, 17 links, 16 joints
Links:
- link link1: geometry collision mesh filename=meshes/uf850/collision/uf850_link1_col_00.stl; collision mesh filename=meshes/uf850/collision/uf850_link1_col_01.stl
- link link2: geometry collision mesh filename=meshes/uf850/collision/uf850_link2_col_00.stl; collision mesh filename=meshes/uf850/collision/uf850_link2_col_01.stl
- link link3: geometry collision mesh filename=meshes/uf850/collision/uf850_link3_col_00.stl; collision mesh filename=meshes/uf850/collision/uf850_link3_col_01.stl
- link link4: geometry collision mesh filename=meshes/uf850/collision/uf850_link4_col_00.stl; collision mesh filename=meshes/uf850/collision/uf850_link4_col_01.stl
- link link5: geometry collision mesh filename=meshes/uf850/collision/uf850_link5_col_00.stl; collision mesh filename=meshes/uf850/collision/uf850_link5_col_01.stl
- link link6: geometry collision mesh filename=meshes/uf850/collision/uf850_link6_col_00.stl; visual mesh filename=meshes/uf850/visual_glb/link6.glb
- link link_base: geometry collision mesh filename=meshes/uf850/collision/uf850_link_base_col_00.stl; collision mesh filename=meshes/uf850/collision/uf850_link_base_col_01.stl

File: assets/urdf/uf850/uf850_visual.glb.urdf (robot description, URDF)
Before this commit: robot gen, 8 links, 7 joints
Links:
- link link1: geometry collision mesh filename=meshes/uf850/collision/uf850_link1_col_00.stl; collision mesh filename=meshes/uf850/collision/uf850_link1_col_01.stl
- link link2: geometry collision mesh filename=meshes/uf850/collision/uf850_link2_col_00.stl; collision mesh filename=meshes/uf850/collision/uf850_link2_col_01.stl
- link link3: geometry collision mesh filename=meshes/uf850/collision/uf850_link3_col_00.stl; collision mesh filename=meshes/uf850/collision/uf850_link3_col_01.stl
- link link4: geometry collision mesh filename=meshes/uf850/collision/uf850_link4_col_00.stl; collision mesh filename=meshes/uf850/collision/uf850_link4_col_01.stl
- link link5: geometry collision mesh filename=meshes/uf850/collision/uf850_link5_col_00.stl; collision mesh filename=meshes/uf850/collision/uf850_link5_col_01.stl
- link link6: geometry collision mesh filename=meshes/uf850/collision/uf850_link6_col_00.stl; visual mesh filename=meshes/uf850/visual_glb/link6.glb
- link link_base: geometry collision mesh filename=meshes/uf850/collision/uf850_link_base_col_00.stl; collision mesh filename=meshes/uf850/collision/uf850_link_base_col_01.stl

File: assets/urdf/xarm5/xarm5_1305.urdf (robot description, URDF)
Before this commit: robot gen, 7 links, 6 joints
Links:
- link link1: geometry collision mesh filename=meshes/xarm5_1305/collision/xarm5_link1_col_00.stl; collision mesh filename=meshes/xarm5_1305/collision/xarm5_link1_col_01.stl
- link link2: geometry collision mesh filename=meshes/xarm5_1305/collision/xarm5_link2_col_00.stl; collision mesh filename=meshes/xarm5_1305/collision/xarm5_link2_col_01.stl
- link link3: geometry collision mesh filename=meshes/xarm5_1305/collision/xarm5_link3_col_00.stl; collision mesh filename=meshes/xarm5_1305/collision/xarm5_link3_col_01.stl
- link link4: geometry collision mesh filename=meshes/xarm5_1305/collision/xarm5_link4_col_00.stl; collision mesh filename=meshes/xarm5_1305/collision/xarm5_link4_col_01.stl
- link link5: geometry collision mesh filename=meshes/xarm5_1305/collision/xarm5_link5_col_00.stl; visual mesh filename=meshes/xarm5_1305/visual/link5.stl
- link link_base: geometry collision mesh filename=meshes/xarm5_1305/collision/xarm5_link_base_col_00.stl; collision mesh filename=meshes/xarm5_1305/collision/xarm5_link_base_col_01.stl

File: assets/urdf/xarm5/xarm5_1305_bio_gripper_g2_movable_visual.glb.urdf (robot description, URDF)
Before this commit: robot xarm5_1305_bio_gripper_g2_movable_visual.glb, 11 links, 10 joints
Links:
- link link1: geometry collision mesh filename=meshes/xarm5_1305/collision/xarm5_link1_col_00.stl; collision mesh filename=meshes/xarm5_1305/collision/xarm5_link1_col_01.stl
- link link2: geometry collision mesh filename=meshes/xarm5_1305/collision/xarm5_link2_col_00.stl; collision mesh filename=meshes/xarm5_1305/collision/xarm5_link2_col_01.stl
- link link3: geometry collision mesh filename=meshes/xarm5_1305/collision/xarm5_link3_col_00.stl; collision mesh filename=meshes/xarm5_1305/collision/xarm5_link3_col_01.stl
- link link4: geometry collision mesh filename=meshes/xarm5_1305/collision/xarm5_link4_col_00.stl; collision mesh filename=meshes/xarm5_1305/collision/xarm5_link4_col_01.stl
- link link5: geometry collision mesh filename=meshes/xarm5_1305/collision/xarm5_link5_col_00.stl; visual mesh filename=meshes/xarm5_1305/visual_glb/link5.glb
- link link_base: geometry collision mesh filename=meshes/xarm5_1305/collision/xarm5_link_base_col_00.stl; collision mesh filename=meshes/xarm5_1305/collision/xarm5_link_base_col_01.stl

File: assets/urdf/xarm5/xarm5_1305_bio_gripper_g2_visual.glb.urdf (robot description, URDF)
Before this commit: robot xarm5_1305_bio_gripper_g2_visual.glb, 12 links, 11 joints
Links:
- link link1: geometry collision mesh filename=meshes/xarm5_1305/collision/xarm5_link1_col_00.stl; collision mesh filename=meshes/xarm5_1305/collision/xarm5_link1_col_01.stl
- link link2: geometry collision mesh filename=meshes/xarm5_1305/collision/xarm5_link2_col_00.stl; collision mesh filename=meshes/xarm5_1305/collision/xarm5_link2_col_01.stl
- link link3: geometry collision mesh filename=meshes/xarm5_1305/collision/xarm5_link3_col_00.stl; collision mesh filename=meshes/xarm5_1305/collision/xarm5_link3_col_01.stl
- link link4: geometry collision mesh filename=meshes/xarm5_1305/collision/xarm5_link4_col_00.stl; collision mesh filename=meshes/xarm5_1305/collision/xarm5_link4_col_01.stl
- link link5: geometry collision mesh filename=meshes/xarm5_1305/collision/xarm5_link5_col_00.stl; visual mesh filename=meshes/xarm5_1305/visual_glb/link5.glb
- link link_base: geometry collision mesh filename=meshes/xarm5_1305/collision/xarm5_link_base_col_00.stl; collision mesh filename=meshes/xarm5_1305/collision/xarm5_link_base_col_01.stl

File: assets/urdf/xarm5/xarm5_1305_g2_movable_visual.urdf (robot description, URDF)
Before this commit: robot xarm5_1305_g2_movable_visual, 15 links, 14 joints
Links:
- link link1: geometry collision mesh filename=meshes/xarm5_1305/collision/xarm5_link1_col_00.stl; collision mesh filename=meshes/xarm5_1305/collision/xarm5_link1_col_01.stl
- link link2: geometry collision mesh filename=meshes/xarm5_1305/collision/xarm5_link2_col_00.stl; collision mesh filename=meshes/xarm5_1305/collision/xarm5_link2_col_01.stl
- link link3: geometry collision mesh filename=meshes/xarm5_1305/collision/xarm5_link3_col_00.stl; collision mesh filename=meshes/xarm5_1305/collision/xarm5_link3_col_01.stl
- link link4: geometry collision mesh filename=meshes/xarm5_1305/collision/xarm5_link4_col_00.stl; collision mesh filename=meshes/xarm5_1305/collision/xarm5_link4_col_01.stl
- link link5: geometry collision mesh filename=meshes/xarm5_1305/collision/xarm5_link5_col_00.stl; visual mesh filename=meshes/xarm5_1305/visual_glb/link5.glb
- link link_base: geometry collision mesh filename=meshes/xarm5_1305/collision/xarm5_link_base_col_00.stl; collision mesh filename=meshes/xarm5_1305/collision/xarm5_link_base_col_01.stl
