Commit message: Update arm collision meshes with selective convex hulls across 5 robots

File: assets/urdf/xarm5/xarm5_1305_g2_visual.urdf (robot description, URDF)
Before this commit: robot xarm5_1305_g2_visual, 16 links, 15 joints
Links:
- link link1: geometry collision mesh filename=meshes/xarm5_1305/collision/xarm5_link1_col_00.stl; collision mesh filename=meshes/xarm5_1305/collision/xarm5_link1_col_01.stl
- link link2: geometry collision mesh filename=meshes/xarm5_1305/collision/xarm5_link2_col_00.stl; collision mesh filename=meshes/xarm5_1305/collision/xarm5_link2_col_01.stl
- link link3: geometry collision mesh filename=meshes/xarm5_1305/collision/xarm5_link3_col_00.stl; collision mesh filename=meshes/xarm5_1305/collision/xarm5_link3_col_01.stl
- link link4: geometry collision mesh filename=meshes/xarm5_1305/collision/xarm5_link4_col_00.stl; collision mesh filename=meshes/xarm5_1305/collision/xarm5_link4_col_01.stl
- link link5: geometry collision mesh filename=meshes/xarm5_1305/collision/xarm5_link5_col_00.stl; visual mesh filename=meshes/xarm5_1305/visual_glb/link5.glb
- link link_base: geometry collision mesh filename=meshes/xarm5_1305/collision/xarm5_link_base_col_00.stl; collision mesh filename=meshes/xarm5_1305/collision/xarm5_link_base_col_01.stl

File: assets/urdf/xarm5/xarm5_1305_visual.glb.urdf (robot description, URDF)
Before this commit: robot gen, 7 links, 6 joints
Links:
- link link1: geometry collision mesh filename=meshes/xarm5_1305/collision/xarm5_link1_col_00.stl; collision mesh filename=meshes/xarm5_1305/collision/xarm5_link1_col_01.stl
- link link2: geometry collision mesh filename=meshes/xarm5_1305/collision/xarm5_link2_col_00.stl; collision mesh filename=meshes/xarm5_1305/collision/xarm5_link2_col_01.stl
- link link3: geometry collision mesh filename=meshes/xarm5_1305/collision/xarm5_link3_col_00.stl; collision mesh filename=meshes/xarm5_1305/collision/xarm5_link3_col_01.stl
- link link4: geometry collision mesh filename=meshes/xarm5_1305/collision/xarm5_link4_col_00.stl; collision mesh filename=meshes/xarm5_1305/collision/xarm5_link4_col_01.stl
- link link5: geometry collision mesh filename=meshes/xarm5_1305/collision/xarm5_link5_col_00.stl; visual mesh filename=meshes/xarm5_1305/visual_glb/link5.glb
- link link_base: geometry collision mesh filename=meshes/xarm5_1305/collision/xarm5_link_base_col_00.stl; collision mesh filename=meshes/xarm5_1305/collision/xarm5_link_base_col_01.stl
